File: uController.sch (KiCad schematic (older format))
At the start: 15 parts, among them J11 USB_B_Micro, U13 STM32F446RETx, U14 STM14_SW, Y1 16MHz, 8pF

Commit message: Major upgrade
Connections:
- net DRV8835_DIR_A: now also U13.34 (PB13)
- net DRV8835_DIR_B: now also U13.37 (PC6)
- net DRV8835_EN: now also U13.33 (PB12)
- net DRV8835_PWM_A: now also U13.35 (PB14)
- net DRV8835_PWM_B: now also U13.36 (PB15)
- net ENC_L_A: now also U13.59 (PB7)
- net ENC_L_B: now also U13.58 (PB6)
- net ENC_R_A: now also U13.22 (PA6)
- net ENC_R_B: now also U13.23 (PA7)
- net ESP_RX: now also U13.16 (PA2)
- net ESP_TX: now also U13.17 (PA3)
- net IMU_SCL: now also U13.41 (PA8)
- net IMU_SDA: now also U13.40 (PC9)
- net SWDO: now also U13.55 (PB3)
- net VL53L0x_SCL: now also U13.61 (PB8)
- net VL53L0x_SDA: now also U13.62 (PB9)
Changed lines of the file:
@@
 Text HLabel 2050 1700 0    50   Input ~ 0
 ~RESET
-Text HLabel 10950 2550 0    50   Input ~ 0
+Text HLabel 10200 2050 0    50   Input ~ 0
 ~BUTTON_UP
-Text HLabel 10950 2650 0    50   Input ~ 0
+Text HLabel 10200 2150 0    50   Input ~ 0
 ~BUTTON_DOWN
-Text HLabel 10950 2750 0    50   Input ~ 0
+Text HLabel 10200 2250 0    50   Input ~ 0
 ~BUTTON_OK
-Text HLabel 10950 2850 0    50   Output ~ 0
+Text HLabel 6350 4550 2    50   Output ~ 0
 VL53L0x_SCL
-Text HLabel 10950 2950 0    50   BiDi ~ 0
+Text HLabel 6350 4650 2    50   BiDi ~ 0
 VL53L0x_SDA
-Text HLabel 10950 3050 0    50   Output ~ 0
+Text HLabel 10200 2550 0    50   Output ~ 0
 VL53L0x_~XSHUT[1]
-Text HLabel 10950 3150 0    50   Output ~ 0
+Text HLabel 10200 2650 0    50   Output ~ 0
 VL53L0x_~XSHUT[2]
-Text HLabel 10950 3250 0    50   Output ~ 0
+Text HLabel 10200 2750 0    50   Output ~ 0
 VL53L0x_~XSHUT[3]
-Text HLabel 10950 3350 0    50   Input ~ 0
+Text HLabel 6350 4450 2    50   Input ~ 0
 ENC_L_A
-Text HLabel 10950 3450 0    50   Input ~ 0
+Text HLabel 6350 4350 2    50   Input ~ 0
 ENC_L_B
-Text HLabel 10950 3550 0    50   Input ~ 0
+Text HLabel 6350 2650 2    50   Input ~ 0
 ENC_R_A
-Text HLabel 10950 3650 0    50   Input ~ 0
+Text HLabel 6350 2750 2    50   Input ~ 0
 ENC_R_B
-Text HLabel 10950 3750 0    50   BiDi ~ 0
+Text HLabel 3950 4600 0    50   BiDi ~ 0
 IMU_SDA
-Text HLabel 10950 3850 0    50   Output ~ 0
+Text HLabel 6850 2800 2    50   Output ~ 0
 IMU_SCL
-Text HLabel 10950 3950 0    50   Output ~ 0
+Text HLabel 6350 2250 2    50   Output ~ 0
 ESP_RX
-Text HLabel 10950 4050 0    50   Input ~ 0
+Text HLabel 6350 2350 2    50   Input ~ 0
 ESP_TX
-Text HLabel 10950 4150 0    50   Input ~ 0
+Text HLabel 10200 3300 0    50   Input ~ 0
 BATT_VOLTAGE
-Text HLabel 10950 4250 0    50   BiDi ~ 0
+Text HLabel 3950 4500 0    50   BiDi ~ 0
 LCD_SDA
-Text HLabel 10950 4350 0    50   Output ~ 0
+Text HLabel 6850 2900 2    50   Output ~ 0
 LCD_SCL
-Text HLabel 10950 4450 0    50   Output ~ 0
+Text HLabel 10200 3600 0    50   Output ~ 0
 BUZZER
-Text HLabel 10950 4550 0    50   Output ~ 0
+Text HLabel 10200 3700 0    50   Output ~ 0
 ~LED_1
-Text HLabel 10950 4650 0    50   Output ~ 0
+Text HLabel 10200 3800 0    50   Output ~ 0
 ~LED_2
-Text HLabel 10950 4750 0    50   Output ~ 0
+Text HLabel 10200 3900 0    50   Output ~ 0
 ~LED_3
-Text HLabel 10950 4850 0    50   Output ~ 0
+Text HLabel 10200 4000 0    50   Output ~ 0
 ~LED_4
-Text HLabel 10950 4950 0    50   Output ~ 0
+Text HLabel 10200 4100 0    50   Output ~ 0
 ~LED_5
-Text HLabel 10950 5050 0    50   Output ~ 0
+Text HLabel 10200 4200 0    50   Output ~ 0
 ~LED_MOUSE_EYE
-Text HLabel 10950 5150 0    50   Output ~ 0
+Text HLabel 6350 4850 2    50   Output ~ 0
 DRV8835_EN
-Text HLabel 10950 5250 0    50   Output ~ 0
+Text HLabel 6350 4950 2    50   Output ~ 0
 DRV8835_DIR_A
-Text HLabel 10950 5450 0    50   Output ~ 0
+Text HLabel 4750 4250 0    50   Output ~ 0
 DRV8835_DIR_B
-Text HLabel 10950 5350 0    50   Output ~ 0
+Text HLabel 6350 5050 2    50   Output ~ 0
 DRV8835_PWM_A
-Text HLabel 10950 5550 0    50   Output ~ 0
+Text HLabel 6350 5150 2    50   Output ~ 0
 DRV8835_PWM_B
 $Comp
@@
 Wire Wire Line
 	2150 2450 2050 2450
+Text HLabel 10200 2850 0    50   Output ~ 0
+VL53L0x_~XSHUT[4]
+Text HLabel 10200 2950 0    50   Output ~ 0
+VL53L0x_~XSHUT[5]
+Wire Wire Line
+	6250 2650 6350 2650
+Wire Wire Line
+	6250 2750 6350 2750
+Wire Wire Line
+	6350 4350 6250 4350
+Wire Wire Line
+	6350 4450 6250 4450
+Wire Wire Line
+	6350 4550 6250 4550
+Wire Wire Line
+	6250 4650 6350 4650
+Wire Wire Line
+	6250 5050 6350 5050
+Wire Wire Line
+	6250 5150 6350 5150
+Wire Wire Line
+	3950 4550 3950 4500
+Wire Wire Line
+	3950 4550 4850 4550
+Wire Wire Line
+	3950 4600 3950 4550
+Connection ~ 3950 4550
+Wire Wire Line
+	6850 2800 6850 2850
+Wire Wire Line
+	6250 2850 6850 2850
+Connection ~ 6850 2850
+Wire Wire Line
+	6850 2850 6850 2900
+Wire Wire Line
+	6350 2350 6250 2350
+Wire Wire Line
+	6250 2250 6350 2250
+Wire Wire Line
+	4850 4250 4750 4250
+Wire Wire Line
+	6250 4950 6350 4950
+Wire Wire Line
+	6250 4850 6350 4850
+Text Label 6350 4050 0    50   ~ 0
+SWDO
+Wire Wire Line
+	6350 4050 6250 4050
 $EndSCHEMATC

Commit message: Tweaks
Swapped ENC_L and ENC_R pins, changed UART pins for STM32<->ESP connection, connected buzzer, LCD and IMU I2C lines were splitted and connected accordingly, added I2C pullup resistors
Parts:
- added R? (x6): 2K2, Resistor_SMD:R_0402_1005Metric, symbol Device:R_Small
- Y1: symbol Device:Crystal_GND24 -> synermycha-electronics-rescue:Crystal_GND24-Device
Connections:
- net +3V3: now also R?.1, R?.1, R?.1, R?.1, R?.1, R?.1
- net BUZZER: now also U13.17 (PA3)
- net ENC_L_A: now also U13.23 (PA7); no longer U13.59 (PB7)
- net ENC_L_B: now also U13.22 (PA6); no longer U13.58 (PB6)
- net ENC_R_A: now also U13.58 (PB6); no longer U13.22 (PA6)
- net ENC_R_B: now also U13.59 (PB7); no longer U13.23 (PA7)
- net ESP_RX: now also U13.42 (PA9); no longer U13.16 (PA2)
- net ESP_TX: now also U13.43 (PA10); no longer U13.17 (PA3)
- net IMU_SCL: now also R?.2
- net IMU_SDA: now also R?.2
- net VL53L0x_SCL: now also R?.2
- net VL53L0x_SDA: now also R?.2
- net LCD_SCL: now reaches U13.29 (PB10)
- net LCD_SCL: now also R?.2
- net LCD_SDA: now reaches U13.53 (PC12)
- net LCD_SDA: now also R?.2
Changed lines of the file:
@@
 $EndDescr
 $Comp
-L Device:Crystal_GND24 Y1
+L synermycha-electronics-rescue:Crystal_GND24-Device Y1
 U 1 1 5E5FF1B5
 P 3900 3200
@@
 Text HLabel 10200 2250 0    50   Input ~ 0
 ~BUTTON_OK
-Text HLabel 6350 4550 2    50   Output ~ 0
+Text HLabel 7250 4550 2    50   Output ~ 0
 VL53L0x_SCL
-Text HLabel 6350 4650 2    50   BiDi ~ 0
+Text HLabel 8050 4650 2    50   BiDi ~ 0
 VL53L0x_SDA
 Text HLabel 10200 2550 0    50   Output ~ 0
@@
 Text HLabel 10200 2750 0    50   Output ~ 0
 VL53L0x_~XSHUT[3]
+Text HLabel 6350 2750 2    50   Input ~ 0
+ENC_L_A
+Text HLabel 6350 2650 2    50   Input ~ 0
+ENC_L_B
+Text HLabel 6350 4350 2    50   Input ~ 0
+ENC_R_A
 Text HLabel 6350 4450 2    50   Input ~ 0
-ENC_L_A
-Text HLabel 6350 4350 2    50   Input ~ 0
-ENC_L_B
-Text HLabel 6350 2650 2    50   Input ~ 0
-ENC_R_A
-Text HLabel 6350 2750 2    50   Input ~ 0
 ENC_R_B
-Text HLabel 3950 4600 0    50   BiDi ~ 0
+Text HLabel 3700 4550 0    50   BiDi ~ 0
 IMU_SDA
-Text HLabel 6850 2800 2    50   Output ~ 0
+Text HLabel 7050 2850 2    50   Output ~ 0
 IMU_SCL
-Text HLabel 6350 2250 2    50   Output ~ 0
+Text HLabel 6350 2950 2    50   Output ~ 0
 ESP_RX
-Text HLabel 6350 2350 2    50   Input ~ 0
+Text HLabel 6350 3050 2    50   Input ~ 0
 ESP_TX
 Text HLabel 10200 3300 0    50   Input ~ 0
 BATT_VOLTAGE
-Text HLabel 3950 4500 0    50   BiDi ~ 0
+Text HLabel 2900 4850 0    50   BiDi ~ 0
 LCD_SDA
-Text HLabel 6850 2900 2    50   Output ~ 0
+Text HLabel 9000 4750 2    50   Output ~ 0
 LCD_SCL
-Text HLabel 10200 3600 0    50   Output ~ 0
+Text HLabel 6350 2350 2    50   Output ~ 0
 BUZZER
 Text HLabel 10200 3700 0    50   Output ~ 0
@@
 	6350 4450 6250 4450
 Wire Wire Line
-	6350 4550 6250 4550
-Wire Wire Line
-	6250 4650 6350 4650
+	7250 4550 7000 4550
+Wire Wire Line
+	6250 4650 7850 4650
 Wire Wire Line
 	6250 5050 6350 5050
@@
 	6250 5150 6350 5150
 Wire Wire Line
-	3950 4550 3950 4500
-Wire Wire Line
-	3950 4550 4850 4550
-Wire Wire Line
-	3950 4600 3950 4550
-Connection ~ 3950 4550
-Wire Wire Line
-	6850 2800 6850 2850
-Wire Wire Line
-	6250 2850 6850 2850
-Connection ~ 6850 2850
-Wire Wire Line
-	6850 2850 6850 2900
-Wire Wire Line
-	6350 2350 6250 2350
-Wire Wire Line
-	6250 2250 6350 2250
+	6350 3050 6250 3050
+Wire Wire Line
+	6250 2950 6350 2950
 Wire Wire Line
 	4850 4250 4750 4250
@@
 Wire Wire Line
 	6350 4050 6250 4050
+Wire Wire Line
+	6250 2850 6850 2850
+Wire Wire Line
+	6250 4750 8700 4750
+Wire Wire Line
+	4850 4850 3150 4850
+Wire Wire Line
+	6350 2350 6250 2350
+$Comp
+L Device:R_Small R?
+U 1 1 5E662907
+P 3800 4450
+F 0 "R?" H 3859 4496 50  0000 L CNN
+F 1 "2K2" H 3859 4405 50  0000 L CNN
+F 2 "Resistor_SMD:R_0402_1005Metric" H 3800 4450 50  0001 C CNN
+F 3 "~" H 3800 4450 50  0001 C CNN
+	1    3800 4450
+	1    0    0    -1
+$EndComp
+Connection ~ 3800 4550
+Wire Wire Line
+	3800 4550 3700 4550
+$Comp
+L power:+3V3 #PWR?
+U 1 1 5E673825
+P 3800 4350
+F 0 "#PWR?" H 3800 4200 50  0001 C CNN
+F 1 "+3V3" H 3815 4523 50  0000 C CNN
+F 2 "" H 3800 4350 50  0001 C CNN
+F 3 "" H 3800 4350 50  0001 C CNN
+	1    3800 4350
+	1    0    0    -1
+$EndComp
+Wire Wire Line
+	3800 4550 4850 4550
+$Comp
+L Device:R_Small R?
+U 1 1 5E6788B6
+P 3150 4750
+F 0 "R?" H 3209 4796 50  0000 L CNN
+F 1 "2K2" H 3209 4705 50  0000 L CNN
+F 2 "Resistor_SMD:R_0402_1005Metric" H 3150 4750 50  0001 C CNN
+F 3 "~" H 3150 4750 50  0001 C CNN
+	1    3150 4750
+	1    0    0    -1
+$EndComp
+Connection ~ 3150 4850
+Wire Wire Line
+	3150 4850 2900 4850
+$Comp
+L power:+3V3 #PWR?
+U 1 1 5E678A77
+P 3150 4650
+F 0 "#PWR?" H 3150 4500 50  0001 C CNN
+F 1 "+3V3" H 3165 4823 50  0000 C CNN
+F 2 "" H 3150 4650 50  0001 C CNN
+F 3 "" H 3150 4650 50  0001 C CNN
+	1    3150 4650
+	1    0    0    -1
+$EndComp
+$Comp
+L Device:R_Small R?
+U 1 1 5E68DC8F
+P 7000 4450
+F 0 "R?" H 7059 4496 50  0000 L CNN
+F 1 "2K2" H 7059 4405 50  0000 L CNN
+F 2 "Resistor_SMD:R_0402_1005Metric" H 7000 4450 50  0001 C CNN
+F 3 "~" H 7000 4450 50  0001 C CNN
+	1    7000 4450
+	1    0    0    -1
+$EndComp
+Connection ~ 7000 4550
+Wire Wire Line
+	7000 4550 6250 4550
+$Comp
+L Device:R_Small R?
+U 1 1 5E68E3C7
+P 7850 4550
+F 0 "R?" H 7909 4596 50  0000 L CNN
+F 1 "2K2" H 7909 4505 50  0000 L CNN
+F 2 "Resistor_SMD:R_0402_1005Metric" H 7850 4550 50  0001 C CNN
+F 3 "~" H 7850 4550 50  0001 C CNN
+	1    7850 4550
+	1    0    0    -1
+$EndComp
+Connection ~ 7850 4650
+Wire Wire Line
+	7850 4650 8050 4650
+$Comp
+L Device:R_Small R?
+U 1 1 5E68E823
+P 8700 4650
+F 0 "R?" H 8759 4696 50  0000 L CNN
+F 1 "2K2" H 8759 4605 50  0000 L CNN
+F 2 "Resistor_SMD:R_0402_1005Metric" H 8700 4650 50  0001 C CNN
+F 3 "~" H 8700 4650 50  0001 C CNN
+	1    8700 4650
+	1    0    0    -1
+$EndComp
+Connection ~ 8700 4750
+Wire Wire Line
+	8700 4750 9000 4750
+$Comp
+L power:+3V3 #PWR?
+U 1 1 5E695E10
+P 7000 4350
+F 0 "#PWR?" H 7000 4200 50  0001 C CNN
+F 1 "+3V3" H 7015 4523 50  0000 C CNN
+F 2 "" H 7000 4350 50  0001 C CNN
+F 3 "" H 7000 4350 50  0001 C CNN
+	1    7000 4350
+	1    0    0    -1
+$EndComp
+$Comp
+L power:+3V3 #PWR?
+U 1 1 5E696677
+P 7850 4450
+F 0 "#PWR?" H 7850 4300 50  0001 C CNN
+F 1 "+3V3" H 7865 4623 50  0000 C CNN
+F 2 "" H 7850 4450 50  0001 C CNN
+F 3 "" H 7850 4450 50  0001 C CNN
+	1    7850 4450
+	1    0    0    -1
+$EndComp
+$Comp
+L power:+3V3 #PWR?
+U 1 1 5E6969D2
+P 8700 4550
+F 0 "#PWR?" H 8700 4400 50  0001 C CNN
+F 1 "+3V3" H 8715 4723 50  0000 C CNN
+F 2 "" H 8700 4550 50  0001 C CNN
+F 3 "" H 8700 4550 50  0001 C CNN
+	1    8700 4550
+	1    0    0    -1
+$EndComp
+$Comp
+L Device:R_Small R?
+U 1 1 5E69B9AF
+P 6850 2750
+F 0 "R?" H 6909 2796 50  0000 L CNN
+F 1 "2K2" H 6909 2705 50  0000 L CNN
+F 2 "Resistor_SMD:R_0402_1005Metric" H 6850 2750 50  0001 C CNN
+F 3 "~" H 6850 2750 50  0001 C CNN
+	1    6850 2750
+	1    0    0    -1
+$EndComp
+Connection ~ 6850 2850
+Wire Wire Line
+	6850 2850 7050 2850
+$Comp
+L power:+3V3 #PWR?
+U 1 1 5E69C5D9
+P 6850 2650
+F 0 "#PWR?" H 6850 2500 50  0001 C CNN
+F 1 "+3V3" H 6865 2823 50  0000 C CNN
+F 2 "" H 6850 2650 50  0001 C CNN
+F 3 "" H 6850 2650 50  0001 C CNN
+	1    6850 2650
+	1    0    0    -1
+$EndComp
 $EndSCHEMATC

Commit message: Many updates
Added 3V3<->2V8 conversion for VC53L0x and leds for XSHUT of those. PCB update
Parts:
- added C37: 10uF, Capacitor_SMD:C_0603_1608Metric, symbol Device:C_Small
- added D?: YELLOW, symbol Device:LED_Small
- added Q5, Q6: Q_NMOS_GDS, Package_TO_SOT_SMD:SOT-23, symbol Device:Q_NMOS_GDS
- added R34, R35: 2K2, Resistor_SMD:R_0402_1005Metric, symbol Device:R_Small
- added R36, R37, R38, R39, R40, R?: 1K, Resistor_SMD:R_0402_1005Metric, symbol Device:R_Small
- added R41, R42, R43, R44, R45: 47K, Resistor_SMD:R_0402_1005Metric, symbol Device:R_Small
- gave numbers to parts that had none: 6
Connections:
- net labels added: +2V8
- wire segments 100 -> 130
Other:
- moved on the sheet: R30, R31, R32

Commit message: uC sch update
Parts:
- added D16, D17, D18, D19: YELLOW, LED_SMD:LED_0402_1005Metric, symbol Device:LED_Small
- added R47, R48, R49, R50: 1K, Resistor_SMD:R_0402_1005Metric, symbol Device:R_Small
- D15: renamed from D?; footprint (none) -> LED_SMD:LED_0402_1005Metric
- gave numbers to parts that had none: 1
Connections:
- wire segments 130 -> 138
Other:
- moved on the sheet: D15, R36, R37, R38, R39, R40, R41, R42, R43, R44, R45, R46

Commit message: Adjusted connections, wiring almost finished
Changed lines of the file:
@@
 Wire Wire Line
 	3900 3050 3900 2950
-Connection ~ 3900 3050
 Wire Wire Line
 	3900 3350 3900 3450
-Connection ~ 3900 3350
 $Comp
 L Device:C_Small C30
