File: uController.sch (KiCad schematic (older format))
At the start: 46 parts, among them J11 USB_B_Micro, Q5 Q_NMOS_GDS, Q6 Q_NMOS_GDS, U13 STM32F446RETx, U14 STM14_SW, Y1 16MHz, 8pF

Commit message: Replaced crystal symbol
Parts:
- removed Y1: 16MHz, 8pF, Crystal:Crystal_SMD_Abracon_ABM8G-4Pin_3.2x2.5mm, symbol synermycha-electronics-rescue:Crystal_GND24-Device
- added Y1: 16Mhz, 8pF, Crystal:Crystal_SMD_Abracon_ABM8G-4Pin_3.2x2.5mm, symbol Device:Crystal_GND24
Changed lines of the file:
@@
 $EndDescr
-$Comp
-L synermycha-electronics-rescue:Crystal_GND24-Device Y1
-U 1 1 5E5FF1B5
-P 3900 3200
-F 0 "Y1" V 3854 3331 50  0000 L CNN
-F 1 "16MHz, 8pF" V 3945 3331 50  0000 L CNN
-F 2 "Crystal:Crystal_SMD_Abracon_ABM8G-4Pin_3.2x2.5mm" H 3900 3200 50  0001 C CNN
-F 3 "~" H 3900 3200 50  0001 C CNN
-	1    3900 3200
-	0    1    1    0
-$EndComp
 $Comp
 L MCU_ST_STM32F4:STM32F446RETx U13
@@
 	1    0    0    -1
 $EndComp
+$Comp
+L Device:Crystal_GND24 Y1
+U 1 1 5E6F9688
+P 3900 3200
+F 0 "Y1" V 3854 3330 50  0000 L CNN
+F 1 "16Mhz, 8pF" V 3945 3330 50  0000 L CNN
+F 2 "Crystal:Crystal_SMD_Abracon_ABM8G-4Pin_3.2x2.5mm" H 3900 3200 50  0001 C CNN
+F 3 "~" H 3900 3200 50  0001 C CNN
+	1    3900 3200
+	0    1    1    0
+$EndComp
+Connection ~ 3900 3050
+Connection ~ 3900 3350
 $EndSCHEMATC

Commit message: Wired all electronics
Connections:
- net labels added: ~LED_6
- wire segments 138 -> 158
Other:
- moved on the sheet: D15, D16, D17, D18, D19, J11, R13, R36, R37, R38, R39, R40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

Commit message: Added connection to RGB for STM32, remapped some pins
Connections:
- net labels added: WS2812B_IN
- wire segments 158 -> 161
Other:
- moved on the sheet: D17, R38, R43, R48
Changed lines of the file:
@@
 Text HLabel 2650 3450 0    50   Output ~ 0
 VL53L0x_~XSHUT[2]
-Text HLabel 8200 2550 2    50   Output ~ 0
+Text HLabel 2650 4100 0    50   Output ~ 0
 VL53L0x_~XSHUT[3]
 Text HLabel 6350 2750 2    50   Input ~ 0
@@
 L Device:R_Small R38
 U 1 1 5E83E376
-P 8000 2550
-F 0 "R38" V 7804 2550 50  0000 C CNN
-F 1 "1K" V 7895 2550 50  0000 C CNN
-F 2 "Resistor_SMD:R_0402_1005Metric" H 8000 2550 50  0001 C CNN
-F 3 "~" H 8000 2550 50  0001 C CNN
-	1    8000 2550
-	0    1    1    0
+P 2850 4100
+F 0 "R38" V 2654 4100 50  0000 C CNN
+F 1 "1K" V 2745 4100 50  0000 C CNN
+F 2 "Resistor_SMD:R_0402_1005Metric" H 2850 4100 50  0001 C CNN
+F 3 "~" H 2850 4100 50  0001 C CNN
+	1    2850 4100
+	0    -1   1    0
 $EndComp
 $Comp
 L Device:R_Small R43
 U 1 1 5E83E37C
-P 8150 2400
-F 0 "R43" H 8209 2446 50  0000 L CNN
-F 1 "47K" H 8209 2355 50  0000 L CNN
-F 2 "Resistor_SMD:R_0402_1005Metric" H 8150 2400 50  0001 C CNN
-F 3 "~" H 8150 2400 50  0001 C CNN
-	1    8150 2400
-	1    0    0    -1
-$EndComp
-Wire Wire Line
-	8200 2550 8150 2550
-Wire Wire Line
-	8150 2550 8150 2500
-Connection ~ 8150 2550
-Wire Wire Line
-	8150 2550 8100 2550
+P 2700 3950
+F 0 "R43" H 2759 3996 50  0000 L CNN
+F 1 "47K" H 2759 3905 50  0000 L CNN
+F 2 "Resistor_SMD:R_0402_1005Metric" H 2700 3950 50  0001 C CNN
+F 3 "~" H 2700 3950 50  0001 C CNN
+	1    2700 3950
+	-1   0    0    -1
+$EndComp
+Wire Wire Line
+	2650 4100 2700 4100
+Wire Wire Line
+	2700 4100 2700 4050
+Connection ~ 2700 4100
+Wire Wire Line
+	2700 4100 2750 4100
 $Comp
 L power:+2V8 #PWR0224
 U 1 1 5E83E386
-P 8150 2300
-F 0 "#PWR0224" H 8150 2150 50  0001 C CNN
-F 1 "+2V8" H 8165 2473 50  0000 C CNN
-F 2 "" H 8150 2300 50  0001 C CNN
-F 3 "" H 8150 2300 50  0001 C CNN
-	1    8150 2300
-	1    0    0    -1
+P 2700 3850
+F 0 "#PWR0224" H 2700 3700 50  0001 C CNN
+F 1 "+2V8" H 2715 4023 50  0000 C CNN
+F 2 "" H 2700 3850 50  0001 C CNN
+F 3 "" H 2700 3850 50  0001 C CNN
+	1    2700 3850
+	-1   0    0    -1
 $EndComp
 $Comp
@@
 L Device:LED_Small D17
 U 1 1 5E8ADCB8
-P 7850 2450
-F 0 "D17" V 7800 2300 50  0000 L CNN
-F 1 "YELLOW" V 7900 2100 50  0000 L CNN
-F 2 "LED_SMD:LED_0402_1005Metric" V 7850 2450 50  0001 C CNN
-F 3 "~" V 7850 2450 50  0001 C CNN
-	1    7850 2450
-	0    1    1    0
-$EndComp
-Wire Wire Line
-	7900 2550 7850 2550
-Connection ~ 7850 2550
+P 3000 4000
+F 0 "D17" V 2950 3850 50  0000 L CNN
+F 1 "YELLOW" V 3050 3650 50  0000 L CNN
+F 2 "LED_SMD:LED_0402_1005Metric" V 3000 4000 50  0001 C CNN
+F 3 "~" V 3000 4000 50  0001 C CNN
+	1    3000 4000
+	0    -1   1    0
+$EndComp
+Wire Wire Line
+	2950 4100 3000 4100
+Connection ~ 3000 4100
 $Comp
 L Device:R_Small R48
 U 1 1 5E8ADCC1
-P 7850 2250
-F 0 "R48" H 7791 2204 50  0000 R CNN
-F 1 "1K" H 7791 2295 50  0000 R CNN
-F 2 "Resistor_SMD:R_0402_1005Metric" H 7850 2250 50  0001 C CNN
-F 3 "~" H 7850 2250 50  0001 C CNN
-	1    7850 2250
-	-1   0    0    1
+P 3000 3800
+F 0 "R48" H 2941 3754 50  0000 R CNN
+F 1 "1K" H 2941 3845 50  0000 R CNN
+F 2 "Resistor_SMD:R_0402_1005Metric" H 3000 3800 50  0001 C CNN
+F 3 "~" H 3000 3800 50  0001 C CNN
+	1    3000 3800
+	1    0    0    1
 $EndComp
 $Comp
 L power:+3V3 #PWR0230
 U 1 1 5E8ADCC7
-P 7850 2150
-F 0 "#PWR0230" H 7850 2000 50  0001 C CNN
-F 1 "+3V3" H 7865 2323 50  0000 C CNN
-F 2 "" H 7850 2150 50  0001 C CNN
-F 3 "" H 7850 2150 50  0001 C CNN
-	1    7850 2150
-	1    0    0    -1
+P 3000 3700
+F 0 "#PWR0230" H 3000 3550 50  0001 C CNN
+F 1 "+3V3" H 3015 3873 50  0000 C CNN
+F 2 "" H 3000 3700 50  0001 C CNN
+F 3 "" H 3000 3700 50  0001 C CNN
+	1    3000 3700
+	-1   0    0    -1
 $EndComp
 $Comp
@@
 	3500 3450 3500 3800
 Wire Wire Line
-	6250 2550 7850 2550
-Wire Wire Line
 	4850 5050 4250 5050
 Wire Wire Line
@@
 Wire Wire Line
 	7400 1850 7850 1850
+Text HLabel 6350 4250 2    50   Output ~ 0
+WS2812B_IN
+Wire Wire Line
+	4850 4050 3500 4050
+Wire Wire Line
+	3500 4050 3500 4100
+Wire Wire Line
+	3500 4100 3000 4100
+Wire Wire Line
+	6350 4250 6250 4250
 $EndSCHEMATC

Commit message: Minor changes in pinout and layout
Parts:
- Y1: symbol Device:Crystal_GND24 -> synermycha-electronics-rescue:Crystal_GND24-Device
Changed lines of the file:
@@
 $EndComp
 $Comp
-L Device:Crystal_GND24 Y1
+L synermycha-electronics-rescue:Crystal_GND24-Device Y1
 U 1 1 5E6F9688
 P 3900 3200
+AR Path="/5E6F9688" Ref="Y1"  Part="1"
+AR Path="/5E5F551F/5E6F9688" Ref="Y1"  Part="1"
 F 0 "Y1" V 3854 3330 50  0000 L CNN
 F 1 "16Mhz, 8pF" V 3945 3330 50  0000 L CNN

Commit message: Minor update in pin connections
Connected Mouse eye led to PWM output
Parts:
- removed Q5, Q6: Q_NMOS_GDS, Package_TO_SOT_SMD:SOT-23, symbol Device:Q_NMOS_GDS
- added Q5, Q6: IRLML2060TRPBF, Package_TO_SOT_SMD:SOT-23, symbol Device:Q_NMOS_GSD
- R11, R12, R13, R30, R31, R32, R34, R35: value 2K2 -> 10K
Connections:
- net +2V8: now also Q5.1 (G), Q6.1 (G)
- net VL53L0x_SCL: now also Q5.2 (S)
- net VL53L0x_SDA: now also Q6.2 (S)
- net ~LED_MOUSE_EYE: now also U13.16 (PA2); no longer U13.20 (PA4)
- net at D18.2 (A), R39.2: now also U13.21 (PA5); no longer U13.16 (PA2)
- net at R32.2, U13.61 (PB8): now also Q5.3 (D)
- net at R31.2, U13.62 (PB9): now also Q6.3 (D)
Changed lines of the file:
@@
 Text HLabel 4750 5150 0    50   Output ~ 0
 ~LED_5
-Text HLabel 6350 2450 2    50   Output ~ 0
+Text HLabel 6350 2250 2    50   Output ~ 0
 ~LED_MOUSE_EYE
 Text HLabel 6350 4850 2    50   Output ~ 0
@@
 P 3800 4450
 F 0 "R12" H 3859 4496 50  0000 L CNN
-F 1 "2K2" H 3859 4405 50  0000 L CNN
+F 1 "10K" H 3859 4405 50  0000 L CNN
 F 2 "Resistor_SMD:R_0402_1005Metric" H 3800 4450 50  0001 C CNN
 F 3 "~" H 3800 4450 50  0001 C CNN
@@
 P 3150 4750
 F 0 "R11" H 3209 4796 50  0000 L CNN
-F 1 "2K2" H 3209 4705 50  0000 L CNN
+F 1 "10K" H 3209 4705 50  0000 L CNN
 F 2 "Resistor_SMD:R_0402_1005Metric" H 3150 4750 50  0001 C CNN
 F 3 "~" H 3150 4750 50  0001 C CNN
@@
 P 6850 4400
 F 0 "R30" H 6909 4446 50  0000 L CNN
-F 1 "2K2" H 6909 4355 50  0000 L CNN
+F 1 "10K" H 6909 4355 50  0000 L CNN
 F 2 "Resistor_SMD:R_0402_1005Metric" H 6850 4400 50  0001 C CNN
 F 3 "~" H 6850 4400 50  0001 C CNN
@@
 P 7250 2750
 F 0 "R13" H 7309 2796 50  0000 L CNN
-F 1 "2K2" H 7309 2705 50  0000 L CNN
+F 1 "10K" H 7309 2705 50  0000 L CNN
 F 2 "Resistor_SMD:R_0402_1005Metric" H 7250 2750 50  0001 C CNN
 F 3 "~" H 7250 2750 50  0001 C CNN
@@
 P 8700 4350
 F 0 "R35" H 8759 4396 50  0000 L CNN
-F 1 "2K2" H 8759 4305 50  0000 L CNN
+F 1 "10K" H 8759 4305 50  0000 L CNN
 F 2 "Resistor_SMD:R_0402_1005Metric" H 8700 4350 50  0001 C CNN
 F 3 "~" H 8700 4350 50  0001 C CNN
@@
 P 8400 4350
 F 0 "R34" H 8459 4396 50  0000 L CNN
-F 1 "2K2" H 8459 4305 50  0000 L CNN
+F 1 "10K" H 8459 4305 50  0000 L CNN
 F 2 "Resistor_SMD:R_0402_1005Metric" H 8400 4350 50  0001 C CNN
 F 3 "~" H 8400 4350 50  0001 C CNN
@@
 $EndComp
 $Comp
-L Device:Q_NMOS_GDS Q6
-U 1 1 5E70F8D9
-P 8150 4550
-F 0 "Q6" V 8399 4550 50  0000 C CNN
-F 1 "Q_NMOS_GDS" V 8490 4550 50  0000 C CNN
-F 2 "Package_TO_SOT_SMD:SOT-23" H 8350 4650 50  0001 C CNN
-F 3 "~" H 8150 4550 50  0001 C CNN
-	1    8150 4550
-	0    -1   1    0
-$EndComp
-$Comp
 L power:+2V8 #PWR0221
 U 1 1 5E724AFB
@@
 $EndComp
 $Comp
-L Device:Q_NMOS_GDS Q5
-U 1 1 5E70D814
-P 7800 4450
-F 0 "Q5" V 8049 4450 50  0000 C CNN
-F 1 "Q_NMOS_GDS" V 8140 4450 50  0000 C CNN
-F 2 "Package_TO_SOT_SMD:SOT-23" H 8000 4550 50  0001 C CNN
-F 3 "~" H 7800 4450 50  0001 C CNN
-	1    7800 4450
-	0    -1   1    0
-$EndComp
-$Comp
 L power:+3V3 #PWR0216
 U 1 1 5E6969D2
@@
 P 7450 4400
 F 0 "R32" H 7509 4446 50  0000 L CNN
-F 1 "2K2" H 7509 4355 50  0000 L CNN
+F 1 "10K" H 7509 4355 50  0000 L CNN
 F 2 "Resistor_SMD:R_0402_1005Metric" H 7450 4400 50  0001 C CNN
 F 3 "~" H 7450 4400 50  0001 C CNN
@@
 P 7150 4400
 F 0 "R31" H 7209 4446 50  0000 L CNN
-F 1 "2K2" H 7209 4355 50  0000 L CNN
+F 1 "10K" H 7209 4355 50  0000 L CNN
 F 2 "Resistor_SMD:R_0402_1005Metric" H 7150 4400 50  0001 C CNN
 F 3 "~" H 7150 4400 50  0001 C CNN
@@
 Connection ~ 3900 3350
 Wire Wire Line
-	6250 2450 6350 2450
-Wire Wire Line
 	7600 3150 8450 3150
 Wire Wire Line
@@
 	2500 5550 3250 5550
 Wire Wire Line
-	6250 2250 7400 2250
-Wire Wire Line
-	7400 2250 7400 1850
-Wire Wire Line
 	7400 1850 7850 1850
 Text HLabel 6350 4250 2    50   Output ~ 0
@@
 Wire Wire Line
 	6350 4250 6250 4250
+$Comp
+L Device:Q_NMOS_GSD Q6
+U 1 1 5E7DEA71
+P 8150 4550
+F 0 "Q6" V 8401 4550 50  0000 C CNN
+F 1 "IRLML2060TRPBF" V 8492 4550 50  0000 C CNN
+F 2 "Package_TO_SOT_SMD:SOT-23" H 8350 4650 50  0001 C CNN
+F 3 "~" H 8150 4550 50  0001 C CNN
+	1    8150 4550
+	0    -1   1    0
+$EndComp
+$Comp
+L Device:Q_NMOS_GSD Q5
+U 1 1 5E7E2296
+P 7800 4450
+F 0 "Q5" V 8051 4450 50  0000 C CNN
+F 1 "IRLML2060TRPBF" V 8142 4450 50  0000 C CNN
+F 2 "Package_TO_SOT_SMD:SOT-23" H 8000 4550 50  0001 C CNN
+F 3 "~" H 7800 4450 50  0001 C CNN
+	1    7800 4450
+	0    -1   1    0
+$EndComp
+Wire Wire Line
+	6250 2550 7100 2550
+Wire Wire Line
+	7100 2550 7100 2350
+Wire Wire Line
+	7100 2350 7400 2350
+Wire Wire Line
+	7400 1850 7400 2350
+Wire Wire Line
+	6250 2250 6350 2250
 $EndSCHEMATC

Commit message: Pinout matching with cube_mx
Connections:
- net at U13.20 (PA4): now also D18.2 (A), R39.2
- now unconnected: U13.21 (PA5)
- no-connect marks 2 -> 3
Other:
- note added: "UNUSED_SPI1_SCK"
- moved on the sheet: C35, R19
Changed lines of the file:
@@
 L Device:C_Small C35
 U 1 1 5E630928
-P 4700 2550
-F 0 "C35" H 4608 2504 50  0000 R CNN
-F 1 "2.2uF" H 4608 2595 50  0000 R CNN
-F 2 "Capacitor_SMD:C_0603_1608Metric" H 4700 2550 50  0001 C CNN
-F 3 "~" H 4700 2550 50  0001 C CNN
-	1    4700 2550
+P 4650 2550
+F 0 "C35" H 4558 2504 50  0000 R CNN
+F 1 "2.2uF" H 4558 2595 50  0000 R CNN
+F 2 "Capacitor_SMD:C_0603_1608Metric" H 4650 2550 50  0001 C CNN
+F 3 "~" H 4650 2550 50  0001 C CNN
+	1    4650 2550
 	-1   0    0    1
 $EndComp
@@
 L Device:R_Small R19
 U 1 1 5E6321B0
-P 4500 2350
-F 0 "R19" H 4559 2396 50  0000 L CNN
-F 1 "10K" H 4559 2305 50  0000 L CNN
-F 2 "Resistor_SMD:R_0402_1005Metric" H 4500 2350 50  0001 C CNN
-F 3 "~" H 4500 2350 50  0001 C CNN
-	1    4500 2350
+P 4450 2350
+F 0 "R19" H 4509 2396 50  0000 L CNN
+F 1 "10K" H 4509 2305 50  0000 L CNN
+F 2 "Resistor_SMD:R_0402_1005Metric" H 4450 2350 50  0001 C CNN
+F 3 "~" H 4450 2350 50  0001 C CNN
+	1    4450 2350
 	1    0    0    -1
 $EndComp
@@
 L power:GND #PWR0149
 U 1 1 5E633AFC
-P 4500 2450
-F 0 "#PWR0149" H 4500 2200 50  0001 C CNN
-F 1 "GND" H 4505 2277 50  0000 C CNN
-F 2 "" H 4500 2450 50  0001 C CNN
-F 3 "" H 4500 2450 50  0001 C CNN
-	1    4500 2450
+P 4450 2450
+F 0 "#PWR0149" H 4450 2200 50  0001 C CNN
+F 1 "GND" H 4455 2277 50  0000 C CNN
+F 2 "" H 4450 2450 50  0001 C CNN
+F 3 "" H 4450 2450 50  0001 C CNN
+	1    4450 2450
 	1    0    0    -1
 $EndComp
@@
 L power:GND #PWR0150
 U 1 1 5E6343F0
-P 4700 2650
-F 0 "#PWR0150" H 4700 2400 50  0001 C CNN
-F 1 "GND" H 4705 2477 50  0000 C CNN
-F 2 "" H 4700 2650 50  0001 C CNN
-F 3 "" H 4700 2650 50  0001 C CNN
-	1    4700 2650
-	1    0    0    -1
-$EndComp
-Wire Wire Line
-	4850 2450 4700 2450
-Wire Wire Line
-	4850 2250 4500 2250
+P 4650 2650
+F 0 "#PWR0150" H 4650 2400 50  0001 C CNN
+F 1 "GND" H 4655 2477 50  0000 C CNN
+F 2 "" H 4650 2650 50  0001 C CNN
+F 3 "" H 4650 2650 50  0001 C CNN
+	1    4650 2650
+	1    0    0    -1
+$EndComp
+Wire Wire Line
+	4850 2450 4650 2450
+Wire Wire Line
+	4850 2250 4450 2250
 Wire Wire Line
 	5350 1850 5350 1800
@@
 Wire Wire Line
 	2500 5550 3250 5550
-Wire Wire Line
-	7400 1850 7850 1850
 Text HLabel 6350 4250 2    50   Output ~ 0
 WS2812B_IN
@@
 $EndComp
 Wire Wire Line
-	6250 2550 7100 2550
-Wire Wire Line
-	7100 2550 7100 2350
-Wire Wire Line
-	7100 2350 7400 2350
-Wire Wire Line
-	7400 1850 7400 2350
-Wire Wire Line
 	6250 2250 6350 2250
+Wire Wire Line
+	6250 2450 7100 2450
+Wire Wire Line
+	7100 2450 7100 1850
+NoConn ~ 6250 2550
+Text Notes 6350 2550 0    50   ~ 0
+UNUSED_SPI1_SCK
+Wire Wire Line
+	7100 1850 7850 1850
 $EndSCHEMATC

Commit message: Issues
Parts:
- R11, R12, R13, R30, R31, R32, R34, R35: value 10K -> 2K7
Connections:
- net at R40.2, U13.2 (PC13): now also D19.1 (K); no longer D19.2 (A)
- net at R39.2, U13.20 (PA4): now also D18.1 (K); no longer D18.2 (A)
- net at R38.2, U13.24 (PC4): now also D17.1 (K); no longer D17.2 (A)
- net at R36.2, U13.3 (PC14): now also D15.1 (K); no longer D15.2 (A)
- net at R37.2, U13.54 (PD2): now also D16.1 (K); no longer D16.2 (A)
- net at R46.1: now also D15.2 (A); no longer D15.1 (K)
- net at R47.1: now also D16.2 (A); no longer D16.1 (K)
- net at R50.1: now also D19.2 (A); no longer D19.1 (K)
- net at R48.1: now also D17.2 (A); no longer D17.1 (K)
- net at R49.1: now also D18.2 (A); no longer D18.1 (K)
Other:
- moved on the sheet: D19
Changed lines of the file:
@@
 P 3800 4450
 F 0 "R12" H 3859 4496 50  0000 L CNN
-F 1 "10K" H 3859 4405 50  0000 L CNN
+F 1 "2K7" H 3859 4405 50  0000 L CNN
 F 2 "Resistor_SMD:R_0402_1005Metric" H 3800 4450 50  0001 C CNN
 F 3 "~" H 3800 4450 50  0001 C CNN
@@
 P 3150 4750
 F 0 "R11" H 3209 4796 50  0000 L CNN
-F 1 "10K" H 3209 4705 50  0000 L CNN
+F 1 "2K7" H 3209 4705 50  0000 L CNN
 F 2 "Resistor_SMD:R_0402_1005Metric" H 3150 4750 50  0001 C CNN
 F 3 "~" H 3150 4750 50  0001 C CNN
@@
 P 6850 4400
 F 0 "R30" H 6909 4446 50  0000 L CNN
-F 1 "10K" H 6909 4355 50  0000 L CNN
+F 1 "2K7" H 6909 4355 50  0000 L CNN
 F 2 "Resistor_SMD:R_0402_1005Metric" H 6850 4400 50  0001 C CNN
 F 3 "~" H 6850 4400 50  0001 C CNN
@@
 P 7250 2750
 F 0 "R13" H 7309 2796 50  0000 L CNN
-F 1 "10K" H 7309 2705 50  0000 L CNN
+F 1 "2K7" H 7309 2705 50  0000 L CNN
 F 2 "Resistor_SMD:R_0402_1005Metric" H 7250 2750 50  0001 C CNN
 F 3 "~" H 7250 2750 50  0001 C CNN
@@
 P 8700 4350
 F 0 "R35" H 8759 4396 50  0000 L CNN
-F 1 "10K" H 8759 4305 50  0000 L CNN
+F 1 "2K7" H 8759 4305 50  0000 L CNN
 F 2 "Resistor_SMD:R_0402_1005Metric" H 8700 4350 50  0001 C CNN
 F 3 "~" H 8700 4350 50  0001 C CNN
@@
 P 8400 4350
 F 0 "R34" H 8459 4396 50  0000 L CNN
-F 1 "10K" H 8459 4305 50  0000 L CNN
+F 1 "2K7" H 8459 4305 50  0000 L CNN
 F 2 "Resistor_SMD:R_0402_1005Metric" H 8400 4350 50  0001 C CNN
 F 3 "~" H 8400 4350 50  0001 C CNN
@@
 P 7450 4400
 F 0 "R32" H 7509 4446 50  0000 L CNN
-F 1 "10K" H 7509 4355 50  0000 L CNN
+F 1 "2K7" H 7509 4355 50  0000 L CNN
 F 2 "Resistor_SMD:R_0402_1005Metric" H 7450 4400 50  0001 C CNN
 F 3 "~" H 7450 4400 50  0001 C CNN
@@
 P 7150 4400
 F 0 "R31" H 7209 4446 50  0000 L CNN
-F 1 "10K" H 7209 4355 50  0000 L CNN
+F 1 "2K7" H 7209 4355 50  0000 L CNN
 F 2 "Resistor_SMD:R_0402_1005Metric" H 7150 4400 50  0001 C CNN
 F 3 "~" H 7150 4400 50  0001 C CNN
@@
 $EndComp
 $Comp
-L Device:R_Small R40
-U 1 1 5E847D5D
-P 2350 5550
-F 0 "R40" V 2154 5550 50  0000 C CNN
-F 1 "1K" V 2245 5550 50  0000 C CNN
-F 2 "Resistor_SMD:R_0402_1005Metric" H 2350 5550 50  0001 C CNN
-F 3 "~" H 2350 5550 50  0001 C CNN
-	1    2350 5550
-	0    -1   1    0
-$EndComp
-$Comp
 L Device:R_Small R45
 U 1 1 5E847D63
@@
 U 1 1 5E8706CE
 P 3900 5650
-F 0 "D15" V 3850 5500 50  0000 L CNN
-F 1 "YELLOW" V 3950 5300 50  0000 L CNN
+F 0 "D15" V 3950 5450 50  0000 L CNN
+F 1 "YELLOW" V 3850 5300 50  0000 L CNN
 F 2 "LED_SMD:LED_0402_1005Metric" V 3900 5650 50  0001 C CNN
 F 3 "~" V 3900 5650 50  0001 C CNN
 	1    3900 5650
-	0    -1   1    0
-$EndComp
-Wire Wire Line
-	3850 5750 3900 5750
-Connection ~ 3900 5750
+	0    -1   -1   0
+$EndComp
 $Comp
 L Device:R_Small R46
@@
 F 3 "~" H 3900 5450 50  0001 C CNN
 	1    3900 5450
-	1    0    0    1
+	-1   0    0    1
 $EndComp
 $Comp
@@
 U 1 1 5E8A288C
 P 3000 3350
-F 0 "D16" V 2950 3200 50  0000 L CNN
-F 1 "YELLOW" V 3050 3000 50  0000 L CNN
+F 0 "D16" V 3050 3150 50  0000 L CNN
+F 1 "YELLOW" V 2950 3000 50  0000 L CNN
 F 2 "LED_SMD:LED_0402_1005Metric" V 3000 3350 50  0001 C CNN
 F 3 "~" V 3000 3350 50  0001 C CNN
 	1    3000 3350
-	0    -1   1    0
-$EndComp
-Wire Wire Line
-	2950 3450 3000 3450
-Connection ~ 3000 3450
+	0    -1   -1   0
+$EndComp
 $Comp
 L Device:R_Small R47
@@
 F 3 "~" H 3000 3150 50  0001 C CNN
 	1    3000 3150
-	1    0    0    1
+	-1   0    0    1
 $EndComp
 $Comp
@@
 $EndComp
 $Comp
-L Device:LED_Small D19
-U 1 1 5E8A7FA3
-P 2500 5450
-F 0 "D19" V 2450 5300 50  0000 L CNN
-F 1 "YELLOW" V 2550 5100 50  0000 L CNN
-F 2 "LED_SMD:LED_0402_1005Metric" V 2500 5450 50  0001 C CNN
-F 3 "~" V 2500 5450 50  0001 C CNN
-	1    2500 5450
-	0    -1   1    0
-$EndComp
-Wire Wire Line
-	2450 5550 2500 5550
-Connection ~ 2500 5550
-$Comp
 L Device:R_Small R50
 U 1 1 5E8A7FAC
@@
 F 3 "~" H 2500 5250 50  0001 C CNN
 	1    2500 5250
-	1    0    0    1
+	-1   0    0    1
 $EndComp
 $Comp
@@
 $EndComp
 $Comp
-L Device:LED_Small D17
-U 1 1 5E8ADCB8
-P 3000 4000
-F 0 "D17" V 2950 3850 50  0000 L CNN
-F 1 "YELLOW" V 3050 3650 50  0000 L CNN
-F 2 "LED_SMD:LED_0402_1005Metric" V 3000 4000 50  0001 C CNN
-F 3 "~" V 3000 4000 50  0001 C CNN
-	1    3000 4000
-	0    -1   1    0
-$EndComp
-Wire Wire Line
-	2950 4100 3000 4100
-Connection ~ 3000 4100
-$Comp
 L Device:R_Small R48
 U 1 1 5E8ADCC1
@@
 F 3 "~" H 3000 3800 50  0001 C CNN
 	1    3000 3800
-	1    0    0    1
+	-1   0    0    1
 $EndComp
 $Comp
@@
 $EndComp
 $Comp
-L Device:LED_Small D18
-U 1 1 5E8B3745
-P 7850 1750
-F 0 "D18" V 7800 1600 50  0000 L CNN
-F 1 "YELLOW" V 7900 1400 50  0000 L CNN
-F 2 "LED_SMD:LED_0402_1005Metric" V 7850 1750 50  0001 C CNN
-F 3 "~" V 7850 1750 50  0001 C CNN
-	1    7850 1750
-	0    1    1    0
-$EndComp
-Wire Wire Line
-	7900 1850 7850 1850
-Connection ~ 7850 1850
-$Comp
 L Device:R_Small R49
 U 1 1 5E8B374E
@@
 F 3 "~" H 7850 1550 50  0001 C CNN
 	1    7850 1550
-	-1   0    0    1
+	1    0    0    1
 $EndComp
 $Comp
@@
 	4050 3800 3500 3800
 Wire Wire Line
-	3000 3450 3500 3450
-Wire Wire Line
 	4050 3450 4850 3450
 Wire Wire Line
@@
 Wire Wire Line
 	4250 5050 4250 5750
-Wire Wire Line
-	3900 5750 4250 5750
 Wire Wire Line
 	4850 4950 3250 4950
@@
 Wire Wire Line
 	6350 2050 6250 2050
-Wire Wire Line
-	2500 5550 3250 5550
 Text HLabel 6350 4250 2    50   Output ~ 0
 WS2812B_IN
@@
 Wire Wire Line
 	3500 4050 3500 4100
-Wire Wire Line
-	3500 4100 3000 4100
 Wire Wire Line
 	6350 4250 6250 4250
@@
 UNUSED_SPI1_SCK
 Wire Wire Line
+	2950 3450 3000 3450
+Connection ~ 3000 3450
+Wire Wire Line
+	3000 3450 3500 3450
+Wire Wire Line
+	2450 5550 2500 5550
+Connection ~ 2500 5550
+Wire Wire Line
+	2500 5550 3250 5550
+Wire Wire Line
+	3850 5750 3900 5750
+Connection ~ 3900 5750
+Wire Wire Line
+	3900 5750 4250 5750
+$Comp
+L Device:LED_Small D19
+U 1 1 5E8A7FA3
+P 2500 5450
+F 0 "D19" V 2550 5550 50  0000 L CNN
+F 1 "YELLOW" V 2450 5550 50  0000 L CNN
+F 2 "LED_SMD:LED_0402_1005Metric" V 2500 5450 50  0001 C CNN
+F 3 "~" V 2500 5450 50  0001 C CNN
+	1    2500 5450
+	0    1    -1   0
+$EndComp
+$Comp
+L Device:R_Small R40
+U 1 1 5E847D5D
+P 2350 5550
+F 0 "R40" V 2154 5550 50  0000 C CNN
+F 1 "1K" V 2245 5550 50  0000 C CNN
+F 2 "Resistor_SMD:R_0402_1005Metric" H 2350 5550 50  0001 C CNN
+F 3 "~" H 2350 5550 50  0001 C CNN
+	1    2350 5550
+	0    -1   1    0
+$EndComp
+Connection ~ 3000 4100
+Wire Wire Line
+	3000 4100 3500 4100
+Wire Wire Line
+	2950 4100 3000 4100
+$Comp
+L Device:LED_Small D17
+U 1 1 5E8ADCB8
+P 3000 4000
+F 0 "D17" V 3050 3800 50  0000 L CNN
+F 1 "YELLOW" V 2950 3650 50  0000 L CNN
+F 2 "LED_SMD:LED_0402_1005Metric" V 3000 4000 50  0001 C CNN
+F 3 "~" V 3000 4000 50  0001 C CNN
+	1    3000 4000
+	0    -1   -1   0
+$EndComp
+Connection ~ 7850 1850
+Wire Wire Line
+	7850 1850 7900 1850
+Wire Wire Line
 	7100 1850 7850 1850
+$Comp
+L Device:LED_Small D18
+U 1 1 5E8B3745
+P 7850 1750
+F 0 "D18" V 7900 1550 50  0000 L CNN
+F 1 "YELLOW" V 7800 1400 50  0000 L CNN
+F 2 "LED_SMD:LED_0402_1005Metric" V 7850 1750 50  0001 C CNN
+F 3 "~" V 7850 1750 50  0001 C CNN
+	1    7850 1750
+	0    1    -1   0
+$EndComp
 $EndSCHEMATC
