File: uController.sch (KiCad schematic (older format))
At the start: 46 parts, among them J11 USB_B_Micro, Q5 IRLML2060TRPBF, Q6 IRLML2060TRPBF, U13 STM32F446RETx, U14 STM14_SW, Y1 16Mhz, 8pF

Commit message: Changes in graphics, added capacitors, changes in xshut
Parts:
- removed R36, R37, R38, R39, R40, R47, R48: 1K, Resistor_SMD:R_0402_1005Metric, symbol Device:R_Small
- removed R41, R44, R45: 47K, Resistor_SMD:R_0402_1005Metric, symbol Device:R_Small
- R42, R43: value 47K -> 140R
- R46, R49, R50: value 1K -> 140R
Connections:
- wire segments 161 -> 147
Other:
- moved on the sheet: D15, D16, D17, D19, R42, R43, R46, R50

Commit message: Estetics
Parts:
- C30, C31: value 8pF -> 18pF
- Y1: value 16Mhz, 8pF -> 16Mhz, 18pF
Changed lines of the file:
@@
 P 3800 2950
 F 0 "C30" V 3571 2950 50  0000 C CNN
-F 1 "8pF" V 3662 2950 50  0000 C CNN
+F 1 "18pF" V 3662 2950 50  0000 C CNN
 F 2 "Capacitor_SMD:C_0402_1005Metric" H 3800 2950 50  0001 C CNN
 F 3 "~" H 3800 2950 50  0001 C CNN
@@
 P 3800 3450
 F 0 "C31" V 3650 3450 50  0000 C CNN
-F 1 "8pF" V 3550 3450 50  0000 C CNN
+F 1 "18pF" V 3550 3450 50  0000 C CNN
 F 2 "Capacitor_SMD:C_0402_1005Metric" H 3800 3450 50  0001 C CNN
 F 3 "~" H 3800 3450 50  0001 C CNN
@@
 AR Path="/5E5F551F/5E6F9688" Ref="Y1"  Part="1"
 F 0 "Y1" V 3854 3330 50  0000 L CNN
-F 1 "16Mhz, 8pF" V 3945 3330 50  0000 L CNN
+F 1 "16Mhz, 18pF" V 3945 3330 50  0000 L CNN
 F 2 "Crystal:Crystal_SMD_Abracon_ABM8G-4Pin_3.2x2.5mm" H 3900 3200 50  0001 C CNN
 F 3 "~" H 3900 3200 50  0001 C CNN

Commit message: Finished encoders, added XSHUT pullups
Parts:
- added R36, R37, R38, R39, R40: 2K7, Resistor_SMD:R_0402_1005Metric, symbol Device:R_Small
Connections:
- wire segments 147 -> 151
Changed lines of the file:
@@
 Wire Wire Line
 	3550 5750 3600 5750
-Wire Wire Line
-	3600 5750 3600 5700
 Connection ~ 3600 5750
 $Comp
@@
 Connection ~ 7850 1850
 Wire Wire Line
-	7100 1850 7850 1850
+	7100 1850 7300 1850
 $Comp
 L Device:LED_Small D18
@@
 $EndComp
 Wire Wire Line
-	2700 3450 3500 3450
-Wire Wire Line
-	2700 4100 3500 4100
-Wire Wire Line
-	2400 5550 3250 5550
+	2700 3450 3100 3450
+Wire Wire Line
+	2700 4100 3100 4100
+Wire Wire Line
+	2400 5550 2800 5550
 Wire Wire Line
 	7850 1850 7900 1850
 Wire Wire Line
-	3600 5750 4250 5750
+	3600 5750 4000 5750
+$Comp
+L Device:R_Small R37
+U 1 1 5E6899C4
+P 3100 3350
+F 0 "R37" H 3159 3396 50  0000 L CNN
+F 1 "2K7" H 3159 3305 50  0000 L CNN
+F 2 "Resistor_SMD:R_0402_1005Metric" H 3100 3350 50  0001 C CNN
+F 3 "~" H 3100 3350 50  0001 C CNN
+	1    3100 3350
+	1    0    0    1
+$EndComp
+Connection ~ 3100 3450
+Wire Wire Line
+	3100 3450 3500 3450
+$Comp
+L power:+2V8 #PWR0228
+U 1 1 5E689D39
+P 3100 3250
+F 0 "#PWR0228" H 3100 3100 50  0001 C CNN
+F 1 "+2V8" H 3115 3423 50  0000 C CNN
+F 2 "" H 3100 3250 50  0001 C CNN
+F 3 "" H 3100 3250 50  0001 C CNN
+	1    3100 3250
+	-1   0    0    -1
+$EndComp
+$Comp
+L Device:R_Small R38
+U 1 1 5E68A2D9
+P 3100 4000
+F 0 "R38" H 3159 4046 50  0000 L CNN
+F 1 "2K7" H 3159 3955 50  0000 L CNN
+F 2 "Resistor_SMD:R_0402_1005Metric" H 3100 4000 50  0001 C CNN
+F 3 "~" H 3100 4000 50  0001 C CNN
+	1    3100 4000
+	1    0    0    1
+$EndComp
+$Comp
+L power:+2V8 #PWR0229
+U 1 1 5E68A2DF
+P 3100 3900
+F 0 "#PWR0229" H 3100 3750 50  0001 C CNN
+F 1 "+2V8" H 3115 4073 50  0000 C CNN
+F 2 "" H 3100 3900 50  0001 C CNN
+F 3 "" H 3100 3900 50  0001 C CNN
+	1    3100 3900
+	-1   0    0    -1
+$EndComp
+$Comp
+L Device:R_Small R36
+U 1 1 5E691B9C
+P 2800 5450
+F 0 "R36" H 2859 5496 50  0000 L CNN
+F 1 "2K7" H 2859 5405 50  0000 L CNN
+F 2 "Resistor_SMD:R_0402_1005Metric" H 2800 5450 50  0001 C CNN
+F 3 "~" H 2800 5450 50  0001 C CNN
+	1    2800 5450
+	1    0    0    1
+$EndComp
+$Comp
+L power:+2V8 #PWR0230
+U 1 1 5E691BA2
+P 2800 5350
+F 0 "#PWR0230" H 2800 5200 50  0001 C CNN
+F 1 "+2V8" H 2815 5523 50  0000 C CNN
+F 2 "" H 2800 5350 50  0001 C CNN
+F 3 "" H 2800 5350 50  0001 C CNN
+	1    2800 5350
+	-1   0    0    -1
+$EndComp
+$Comp
+L Device:R_Small R39
+U 1 1 5E698E1F
+P 4000 5650
+F 0 "R39" H 4059 5696 50  0000 L CNN
+F 1 "2K7" H 4059 5605 50  0000 L CNN
+F 2 "Resistor_SMD:R_0402_1005Metric" H 4000 5650 50  0001 C CNN
+F 3 "~" H 4000 5650 50  0001 C CNN
+	1    4000 5650
+	1    0    0    1
+$EndComp
+$Comp
+L power:+2V8 #PWR0231
+U 1 1 5E698E25
+P 4000 5550
+F 0 "#PWR0231" H 4000 5400 50  0001 C CNN
+F 1 "+2V8" H 4015 5723 50  0000 C CNN
+F 2 "" H 4000 5550 50  0001 C CNN
+F 3 "" H 4000 5550 50  0001 C CNN
+	1    4000 5550
+	-1   0    0    -1
+$EndComp
+$Comp
+L Device:R_Small R40
+U 1 1 5E69FF44
+P 7300 1750
+F 0 "R40" H 7359 1796 50  0000 L CNN
+F 1 "2K7" H 7359 1705 50  0000 L CNN
+F 2 "Resistor_SMD:R_0402_1005Metric" H 7300 1750 50  0001 C CNN
+F 3 "~" H 7300 1750 50  0001 C CNN
+	1    7300 1750
+	1    0    0    1
+$EndComp
+$Comp
+L power:+2V8 #PWR0235
+U 1 1 5E69FF4A
+P 7300 1650
+F 0 "#PWR0235" H 7300 1500 50  0001 C CNN
+F 1 "+2V8" H 7315 1823 50  0000 C CNN
+F 2 "" H 7300 1650 50  0001 C CNN
+F 3 "" H 7300 1650 50  0001 C CNN
+	1    7300 1650
+	-1   0    0    -1
+$EndComp
+Connection ~ 7300 1850
+Wire Wire Line
+	7300 1850 7850 1850
+Connection ~ 2800 5550
+Wire Wire Line
+	2800 5550 3250 5550
+Connection ~ 4000 5750
+Wire Wire Line
+	4000 5750 4250 5750
+Connection ~ 3100 4100
+Wire Wire Line
+	3100 4100 3500 4100
 $EndSCHEMATC

Commit message: Czyszczenie
Usunięto linie 5V oraz 2V8. Poprawiono symbol dla diody RGB
Parts:
- removed J11: USB_B_Micro, Connector_USB:USB_Micro-B_Amphenol_10103594-0001LF_Horizontal, symbol Connector:USB_B_Micro
- removed Q5, Q6: IRLML2060TRPBF, Package_TO_SOT_SMD:SOT-23, symbol Device:Q_NMOS_GSD
- removed R34, R35: 2K7, Resistor_SMD:R_0402_1005Metric, symbol Device:R_Small
- added J4: USB_C_Receptacle, symbol Connector:USB_C_Receptacle
Connections:
- net labels removed: +2V8, STM32_D+, STM32_D-, STM32_VBUS
- wire segments 151 -> 134
- no-connect marks 3 -> 2

Commit message: Zmieniono moduł wifi na bluetooth oraz złącze usb - c
Parts:
- J4: footprint (none) -> Connector_USB:USB_C_Receptacle_GCT_USB4085; symbol Connector:USB_C_Receptacle -> synermycha-electronics-rescue:USB_C_Receptacle-Connector
Changed lines of the file:
@@
 $EndComp
 $Comp
-L Connector:USB_C_Receptacle J4
+L synermycha-electronics-rescue:USB_C_Receptacle-Connector J4
 U 1 1 5F661DD8
 P 10200 3100
+AR Path="/5F661DD8" Ref="J4"  Part="1"
+AR Path="/5E5F551F/5F661DD8" Ref="J4"  Part="1"
 F 0 "J4" H 9770 2889 50  0000 R CNN
 F 1 "USB_C_Receptacle" H 9770 2798 50  0000 R CNN
-F 2 "" H 10350 3100 50  0001 C CNN
+F 2 "Connector_USB:USB_C_Receptacle_GCT_USB4085" H 10350 3100 50  0001 C CNN
 F 3 "https://www.usb.org/sites/default/files/documents/usb_type-c.zip" H 10350 3100 50  0001 C CNN
 	1    10200 3100

Commit message: Holy $hi3t
Parts:
- Y1: footprint Crystal:Crystal_SMD_Abracon_ABM8G-4Pin_3.2x2.5mm -> Crystal:Crystal_SMD_Abracon_ABM10-4Pin_2.5x2.0mm
Connections:
- net +3V3: no longer R42.1, R43.1, R46.2, R49.2, R50.2
- net GND: now also D15.1 (K), D16.1 (K), D17.1 (K), D18.1 (K), D19.1 (K)
- net VL53L0x_~XSHUT[1]: now also R46.2; no longer D15.1 (K)
- net VL53L0x_~XSHUT[2]: now also R42.2; no longer D16.1 (K)
- net VL53L0x_~XSHUT[3]: now also R43.2; no longer D17.1 (K)
- net VL53L0x_~XSHUT[4]: now also R49.2; no longer D18.1 (K)
- net VL53L0x_~XSHUT[5]: now also R50.2; no longer D19.1 (K)
- net ~BUTTON_DOWN: now also U13.50 (PA15); no longer U13.52 (PC11)
- net ~BUTTON_OK: now also U13.52 (PC11); no longer U13.51 (PC10)
- net ~BUTTON_UP: now also U13.51 (PC10); no longer U13.50 (PA15)
- net at D16.2 (A): now also R42.1; no longer R42.2
- net at D17.2 (A): now also R43.1; no longer R43.2
Other:
- moved on the sheet: D15, D16, D17, D18, D19, R42, R43, R46, R49, R50
Changed lines of the file:
@@
 Text HLabel 2050 1700 0    50   Input ~ 0
 ~RESET
+Text HLabel 4750 4650 0    50   Input ~ 0
+~BUTTON_UP
 Text HLabel 6350 3550 2    50   Input ~ 0
-~BUTTON_UP
+~BUTTON_DOWN
 Text HLabel 4750 4750 0    50   Input ~ 0
-~BUTTON_DOWN
-Text HLabel 4750 4650 0    50   Input ~ 0
 ~BUTTON_OK
 Text HLabel 7600 4550 2    50   Output ~ 0
@@
 L Device:R_Small R42
 U 1 1 5E839F84
-P 2700 3150
-F 0 "R42" H 2759 3196 50  0000 L CNN
-F 1 "140R" H 2759 3105 50  0000 L CNN
-F 2 "Resistor_SMD:R_0402_1005Metric" H 2700 3150 50  0001 C CNN
-F 3 "~" H 2700 3150 50  0001 C CNN
-	1    2700 3150
-	-1   0    0    -1
-$EndComp
-Wire Wire Line
-	2650 3450 2700 3450
-Connection ~ 2700 3450
+P 2700 3550
+F 0 "R42" H 2759 3596 50  0000 L CNN
+F 1 "140R" H 2759 3505 50  0000 L CNN
+F 2 "Resistor_SMD:R_0402_1005Metric" H 2700 3550 50  0001 C CNN
+F 3 "~" H 2700 3550 50  0001 C CNN
+	1    2700 3550
+	1    0    0    1
+$EndComp
 $Comp
 L Device:R_Small R43
 U 1 1 5E83E37C
-P 2700 3800
-F 0 "R43" H 2759 3846 50  0000 L CNN
-F 1 "140R" H 2759 3755 50  0000 L CNN
-F 2 "Resistor_SMD:R_0402_1005Metric" H 2700 3800 50  0001 C CNN
-F 3 "~" H 2700 3800 50  0001 C CNN
-	1    2700 3800
-	-1   0    0    -1
-$EndComp
-Wire Wire Line
-	2650 4100 2700 4100
-Connection ~ 2700 4100
+P 2700 4200
+F 0 "R43" H 2759 4246 50  0000 L CNN
+F 1 "140R" H 2759 4155 50  0000 L CNN
+F 2 "Resistor_SMD:R_0402_1005Metric" H 2700 4200 50  0001 C CNN
+F 3 "~" H 2700 4200 50  0001 C CNN
+	1    2700 4200
+	1    0    0    1
+$EndComp
 Wire Wire Line
 	2350 5550 2400 5550
@@
 L Device:LED_Small D15
 U 1 1 5E8706CE
-P 3600 5650
-F 0 "D15" V 3650 5450 50  0000 L CNN
-F 1 "YELLOW" V 3550 5300 50  0000 L CNN
-F 2 "LED_SMD:LED_0402_1005Metric" V 3600 5650 50  0001 C CNN
-F 3 "~" V 3600 5650 50  0001 C CNN
-	1    3600 5650
+P 3600 6050
+F 0 "D15" V 3650 5850 50  0000 L CNN
+F 1 "YELLOW" V 3550 5700 50  0000 L CNN
+F 2 "LED_SMD:LED_0402_1005Metric" V 3600 6050 50  0001 C CNN
+F 3 "~" V 3600 6050 50  0001 C CNN
+	1    3600 6050
 	0    -1   -1   0
 $EndComp
@@
 L Device:R_Small R46
 U 1 1 5E897495
-P 3600 5450
-F 0 "R46" H 3541 5404 50  0000 R CNN
-F 1 "140R" H 3541 5495 50  0000 R CNN
-F 2 "Resistor_SMD:R_0402_1005Metric" H 3600 5450 50  0001 C CNN
-F 3 "~" H 3600 5450 50  0001 C CNN
-	1    3600 5450
+P 3600 5850
+F 0 "R46" H 3541 5804 50  0000 R CNN
+F 1 "140R" H 3541 5895 50  0000 R CNN
+F 2 "Resistor_SMD:R_0402_1005Metric" H 3600 5850 50  0001 C CNN
+F 3 "~" H 3600 5850 50  0001 C CNN
+	1    3600 5850
 	-1   0    0    1
 $EndComp
@@
 L Device:LED_Small D16
 U 1 1 5E8A288C
-P 2700 3350
-F 0 "D16" V 2750 3150 50  0000 L CNN
-F 1 "YELLOW" V 2650 3000 50  0000 L CNN
-F 2 "LED_SMD:LED_0402_1005Metric" V 2700 3350 50  0001 C CNN
-F 3 "~" V 2700 3350 50  0001 C CNN
-	1    2700 3350
+P 2700 3750
+F 0 "D16" V 2750 3550 50  0000 L CNN
+F 1 "YELLOW" V 2650 3400 50  0000 L CNN
+F 2 "LED_SMD:LED_0402_1005Metric" V 2700 3750 50  0001 C CNN
+F 3 "~" V 2700 3750 50  0001 C CNN
+	1    2700 3750
 	0    -1   -1   0
 $EndComp
@@
 L Device:R_Small R50
 U 1 1 5E8A7FAC
-P 2400 5250
-F 0 "R50" H 2341 5204 50  0000 R CNN
-F 1 "140R" H 2341 5295 50  0000 R CNN
-F 2 "Resistor_SMD:R_0402_1005Metric" H 2400 5250 50  0001 C CNN
-F 3 "~" H 2400 5250 50  0001 C CNN
-	1    2400 5250
+P 2400 5650
+F 0 "R50" H 2341 5604 50  0000 R CNN
+F 1 "140R" H 2341 5695 50  0000 R CNN
+F 2 "Resistor_SMD:R_0402_1005Metric" H 2400 5650 50  0001 C CNN
+F 3 "~" H 2400 5650 50  0001 C CNN
+	1    2400 5650
 	-1   0    0    1
 $EndComp
@@
 L Device:R_Small R49
 U 1 1 5E8B374E
-P 7850 1550
-F 0 "R49" H 7791 1504 50  0000 R CNN
-F 1 "140R" H 7791 1595 50  0000 R CNN
-F 2 "Resistor_SMD:R_0402_1005Metric" H 7850 1550 50  0001 C CNN
-F 3 "~" H 7850 1550 50  0001 C CNN
-	1    7850 1550
+P 7850 1950
+F 0 "R49" H 7791 1904 50  0000 R CNN
+F 1 "140R" H 7791 1995 50  0000 R CNN
+F 2 "Resistor_SMD:R_0402_1005Metric" H 7850 1950 50  0001 C CNN
+F 3 "~" H 7850 1950 50  0001 C CNN
+	1    7850 1950
 	1    0    0    1
 $EndComp
@@
 F 0 "Y1" V 3854 3330 50  0000 L CNN
 F 1 "16Mhz, 18pF" V 3945 3330 50  0000 L CNN
-F 2 "Crystal:Crystal_SMD_Abracon_ABM8G-4Pin_3.2x2.5mm" H 3900 3200 50  0001 C CNN
+F 2 "Crystal:Crystal_SMD_Abracon_ABM10-4Pin_2.5x2.0mm" H 3900 3200 50  0001 C CNN
 F 3 "~" H 3900 3200 50  0001 C CNN
 	1    3900 3200
@@
 UNUSED_SPI1_SCK
 $Comp
-L Device:LED_Small D19
-U 1 1 5E8A7FA3
-P 2400 5450
-F 0 "D19" V 2450 5550 50  0000 L CNN
-F 1 "YELLOW" V 2350 5550 50  0000 L CNN
-F 2 "LED_SMD:LED_0402_1005Metric" V 2400 5450 50  0001 C CNN
-F 3 "~" V 2400 5450 50  0001 C CNN
-	1    2400 5450
-	0    1    -1   0
-$EndComp
-$Comp
 L Device:LED_Small D17
 U 1 1 5E8ADCB8
-P 2700 4000
-F 0 "D17" V 2750 3800 50  0000 L CNN
-F 1 "YELLOW" V 2650 3650 50  0000 L CNN
-F 2 "LED_SMD:LED_0402_1005Metric" V 2700 4000 50  0001 C CNN
-F 3 "~" V 2700 4000 50  0001 C CNN
-	1    2700 4000
+P 2700 4400
+F 0 "D17" V 2750 4200 50  0000 L CNN
+F 1 "YELLOW" V 2650 4050 50  0000 L CNN
+F 2 "LED_SMD:LED_0402_1005Metric" V 2700 4400 50  0001 C CNN
+F 3 "~" V 2700 4400 50  0001 C CNN
+	1    2700 4400
 	0    -1   -1   0
 $EndComp
@@
 L Device:LED_Small D18
 U 1 1 5E8B3745
-P 7850 1750
-F 0 "D18" V 7900 1550 50  0000 L CNN
-F 1 "YELLOW" V 7800 1400 50  0000 L CNN
-F 2 "LED_SMD:LED_0402_1005Metric" V 7850 1750 50  0001 C CNN
-F 3 "~" V 7850 1750 50  0001 C CNN
-	1    7850 1750
+P 7850 2150
+F 0 "D18" V 7900 1950 50  0000 L CNN
+F 1 "YELLOW" V 7800 1800 50  0000 L CNN
+F 2 "LED_SMD:LED_0402_1005Metric" V 7850 2150 50  0001 C CNN
+F 3 "~" V 7850 2150 50  0001 C CNN
+	1    7850 2150
 	0    1    -1   0
 $EndComp
-Wire Wire Line
-	2700 3450 3100 3450
-Wire Wire Line
-	2700 4100 3100 4100
 Wire Wire Line
 	2400 5550 2800 5550
@@
 $EndComp
 $Comp
-L power:+3V3 #PWR0135
-U 1 1 5F64A76E
-P 2400 5150
-F 0 "#PWR0135" H 2400 5000 50  0001 C CNN
-F 1 "+3V3" H 2415 5323 50  0000 C CNN
-F 2 "" H 2400 5150 50  0001 C CNN
-F 3 "" H 2400 5150 50  0001 C CNN
-	1    2400 5150
-	1    0    0    -1
-$EndComp
-$Comp
-L power:+3V3 #PWR0136
-U 1 1 5F64ACF3
-P 3600 5350
-F 0 "#PWR0136" H 3600 5200 50  0001 C CNN
-F 1 "+3V3" H 3615 5523 50  0000 C CNN
-F 2 "" H 3600 5350 50  0001 C CNN
-F 3 "" H 3600 5350 50  0001 C CNN
-	1    3600 5350
-	1    0    0    -1
-$EndComp
-$Comp
 L power:+3V3 #PWR0137
 U 1 1 5F64C720
@@
 $EndComp
 $Comp
-L power:+3V3 #PWR0138
-U 1 1 5F64CCEA
-P 2700 3050
-F 0 "#PWR0138" H 2700 2900 50  0001 C CNN
-F 1 "+3V3" H 2715 3223 50  0000 C CNN
-F 2 "" H 2700 3050 50  0001 C CNN
-F 3 "" H 2700 3050 50  0001 C CNN
-	1    2700 3050
-	1    0    0    -1
-$EndComp
-$Comp
-L power:+3V3 #PWR0139
-U 1 1 5F64D2D6
-P 2700 3700
-F 0 "#PWR0139" H 2700 3550 50  0001 C CNN
-F 1 "+3V3" H 2715 3873 50  0000 C CNN
-F 2 "" H 2700 3700 50  0001 C CNN
-F 3 "" H 2700 3700 50  0001 C CNN
-	1    2700 3700
-	1    0    0    -1
-$EndComp
-$Comp
 L power:+3V3 #PWR0140
 U 1 1 5F64D886
@@
 F 3 "" H 7300 1650 50  0001 C CNN
 	1    7300 1650
-	1    0    0    -1
-$EndComp
-$Comp
-L power:+3V3 #PWR0143
-U 1 1 5F658192
-P 7850 1450
-F 0 "#PWR0143" H 7850 1300 50  0001 C CNN
-F 1 "+3V3" H 7865 1623 50  0000 C CNN
-F 2 "" H 7850 1450 50  0001 C CNN
-F 3 "" H 7850 1450 50  0001 C CNN
-	1    7850 1450
 	1    0    0    -1
 $EndComp
@@
 	-1   0    0    -1
 $EndComp
+$Comp
+L Device:LED_Small D19
+U 1 1 5E8A7FA3
+P 2400 5850
+F 0 "D19" V 2450 5950 50  0000 L CNN
+F 1 "YELLOW" V 2350 5950 50  0000 L CNN
+F 2 "LED_SMD:LED_0402_1005Metric" V 2400 5850 50  0001 C CNN
+F 3 "~" V 2400 5850 50  0001 C CNN
+	1    2400 5850
+	0    1    -1   0
+$EndComp
+Wire Wire Line
+	2650 4100 2700 4100
+Connection ~ 2700 4100
+Wire Wire Line
+	2700 4100 3100 4100
+Wire Wire Line
+	2650 3450 2700 3450
+Connection ~ 2700 3450
+Wire Wire Line
+	2700 3450 3100 3450
+$Comp
+L power:GND #PWR0135
+U 1 1 5F7F5F84
+P 2400 5950
+F 0 "#PWR0135" H 2400 5700 50  0001 C CNN
+F 1 "GND" H 2405 5777 50  0000 C CNN
+F 2 "" H 2400 5950 50  0001 C CNN
+F 3 "" H 2400 5950 50  0001 C CNN
+	1    2400 5950
+	1    0    0    -1
+$EndComp
+$Comp
+L power:GND #PWR0136
+U 1 1 5F7F697D
+P 2700 4500
+F 0 "#PWR0136" H 2700 4250 50  0001 C CNN
+F 1 "GND" H 2705 4327 50  0000 C CNN
+F 2 "" H 2700 4500 50  0001 C CNN
+F 3 "" H 2700 4500 50  0001 C CNN
+	1    2700 4500
+	1    0    0    -1
+$EndComp
+$Comp
+L power:GND #PWR0138
+U 1 1 5F7F738B
+P 2700 3850
+F 0 "#PWR0138" H 2700 3600 50  0001 C CNN
+F 1 "GND" H 2705 3677 50  0000 C CNN
+F 2 "" H 2700 3850 50  0001 C CNN
+F 3 "" H 2700 3850 50  0001 C CNN
+	1    2700 3850
+	1    0    0    -1
+$EndComp
+$Comp
+L power:GND #PWR0139
+U 1 1 5F7F8216
+P 7850 2250
+F 0 "#PWR0139" H 7850 2000 50  0001 C CNN
+F 1 "GND" H 7855 2077 50  0000 C CNN
+F 2 "" H 7850 2250 50  0001 C CNN
+F 3 "" H 7850 2250 50  0001 C CNN
+	1    7850 2250
+	1    0    0    -1
+$EndComp
+$Comp
+L power:GND #PWR0143
+U 1 1 5F7FF6EF
+P 3600 6150
+F 0 "#PWR0143" H 3600 5900 50  0001 C CNN
+F 1 "GND" H 3605 5977 50  0000 C CNN
+F 2 "" H 3600 6150 50  0001 C CNN
+F 3 "" H 3600 6150 50  0001 C CNN
+	1    3600 6150
+	1    0    0    -1
+$EndComp
 $EndSCHEMATC
