File: IMU.sch (KiCad schematic (older format))
At the start: 5 parts, among them U12 MPU-9250

Commit message: Issues
Parts:
- added R?: 10K, Resistor_SMD:R_0402_1005Metric, symbol Device:R_Small
Connections:
- net +3V3: now also U12.1 (RESV_VDDIO)
- net GND: now also U12.20 (RESV_GND), R?.1
- net at U12.11 (FSYNC): now also R?.2
- no-connect marks 6 -> 3
Other:
- moved on the sheet: C24, C26
Changed lines of the file:
@@
 L power:+3V3 #PWR?
 U 1 1 5E6F367E
-P 6800 2700
+P 7200 2700
 AR Path="/5E5F55D4/5E6F367E" Ref="#PWR?"  Part="1"
 AR Path="/5E6F1BD7/5E6F367E" Ref="#PWR0174"  Part="1"
-F 0 "#PWR0174" H 6800 2550 50  0001 C CNN
-F 1 "+3V3" H 6815 2873 50  0000 C CNN
-F 2 "" H 6800 2700 50  0001 C CNN
-F 3 "" H 6800 2700 50  0001 C CNN
-	1    6800 2700
+F 0 "#PWR0174" H 7200 2550 50  0001 C CNN
+F 1 "+3V3" H 7215 2873 50  0000 C CNN
+F 2 "" H 7200 2700 50  0001 C CNN
+F 3 "" H 7200 2700 50  0001 C CNN
+	1    7200 2700
 	1    0    0    -1
 $EndComp
@@
 L Device:C_Small C?
 U 1 1 5E6F3684
-P 6400 2800
+P 6800 2800
 AR Path="/5E5F55D4/5E6F3684" Ref="C?"  Part="1"
 AR Path="/5E6F1BD7/5E6F3684" Ref="C24"  Part="1"
-F 0 "C24" H 6492 2846 50  0000 L CNN
-F 1 "0.1uF" H 6492 2755 50  0000 L CNN
-F 2 "Capacitor_SMD:C_0402_1005Metric" H 6400 2800 50  0001 C CNN
-F 3 "~" H 6400 2800 50  0001 C CNN
-	1    6400 2800
+F 0 "C24" H 6892 2846 50  0000 L CNN
+F 1 "0.1uF" H 6892 2755 50  0000 L CNN
+F 2 "Capacitor_SMD:C_0402_1005Metric" H 6800 2800 50  0001 C CNN
+F 3 "~" H 6800 2800 50  0001 C CNN
+	1    6800 2800
 	1    0    0    -1
 $EndComp
@@
 $EndComp
 Wire Wire Line
-	6400 2700 5800 2700
-Wire Wire Line
 	5600 2700 5600 2900
-Connection ~ 6400 2700
+Connection ~ 6800 2700
 Wire Wire Line
 	5800 2900 5800 2700
-Connection ~ 5800 2700
 Wire Wire Line
 	5800 2700 5600 2700
@@
 L power:GND #PWR?
 U 1 1 5E6F369C
-P 6400 2900
+P 7200 2900
 AR Path="/5E5F55D4/5E6F369C" Ref="#PWR?"  Part="1"
 AR Path="/5E6F1BD7/5E6F369C" Ref="#PWR0176"  Part="1"
-F 0 "#PWR0176" H 6400 2650 50  0001 C CNN
-F 1 "GND" H 6405 2727 50  0000 C CNN
-F 2 "" H 6400 2900 50  0001 C CNN
-F 3 "" H 6400 2900 50  0001 C CNN
-	1    6400 2900
+F 0 "#PWR0176" H 7200 2650 50  0001 C CNN
+F 1 "GND" H 7205 2727 50  0000 C CNN
+F 2 "" H 7200 2900 50  0001 C CNN
+F 3 "" H 7200 2900 50  0001 C CNN
+	1    7200 2900
 	1    0    0    -1
 $EndComp
@@
 	1    0    0    -1
 $EndComp
-NoConn ~ 5000 4000
-NoConn ~ 6400 4100
-NoConn ~ 6400 4200
 $Comp
 L Device:C_Small C?
 U 1 1 5E6F36BE
-P 6800 2800
+P 7200 2800
 AR Path="/5E5F55D4/5E6F36BE" Ref="C?"  Part="1"
 AR Path="/5E6F1BD7/5E6F36BE" Ref="C26"  Part="1"
-F 0 "C26" H 6892 2846 50  0000 L CNN
-F 1 "10uF" H 6892 2755 50  0000 L CNN
-F 2 "Capacitor_SMD:C_0603_1608Metric" H 6800 2800 50  0001 C CNN
-F 3 "~" H 6800 2800 50  0001 C CNN
-	1    6800 2800
+F 0 "C26" H 7292 2846 50  0000 L CNN
+F 1 "10uF" H 7292 2755 50  0000 L CNN
+F 2 "Capacitor_SMD:C_0603_1608Metric" H 7200 2800 50  0001 C CNN
+F 3 "~" H 7200 2800 50  0001 C CNN
+	1    7200 2800
 	1    0    0    -1
 $EndComp
@@
 $EndComp
 Wire Wire Line
-	6400 2700 6800 2700
-Connection ~ 6800 2700
+	6800 2700 7200 2700
+Connection ~ 7200 2700
 Wire Wire Line
 	5000 3600 4850 3600
@@
 	1    0    0    -1
 $EndComp
+$Comp
+L Device:R_Small R?
+U 1 1 5E717285
+P 4950 4200
+AR Path="/5E5F55D4/5E717285" Ref="R?"  Part="1"
+AR Path="/5E6F1BD7/5E717285" Ref="R?"  Part="1"
+F 0 "R?" H 4891 4154 50  0000 R CNN
+F 1 "10K" H 4891 4245 50  0000 R CNN
+F 2 "Resistor_SMD:R_0402_1005Metric" H 4950 4200 50  0001 C CNN
+F 3 "~" H 4950 4200 50  0001 C CNN
+	1    4950 4200
+	-1   0    0    1
+$EndComp
+$Comp
+L power:GND #PWR?
+U 1 1 5E717865
+P 4950 4300
+AR Path="/5E5F55D4/5E717865" Ref="#PWR?"  Part="1"
+AR Path="/5E6F1BD7/5E717865" Ref="#PWR?"  Part="1"
+F 0 "#PWR?" H 4950 4050 50  0001 C CNN
+F 1 "GND" H 4955 4127 50  0000 C CNN
+F 2 "" H 4950 4300 50  0001 C CNN
+F 3 "" H 4950 4300 50  0001 C CNN
+	1    4950 4300
+	1    0    0    -1
+$EndComp
+Wire Wire Line
+	5000 4000 4950 4000
+Wire Wire Line
+	4950 4000 4950 4100
+Wire Wire Line
+	6400 4200 6450 4200
+Wire Wire Line
+	6450 4200 6450 4250
+$Comp
+L power:GND #PWR?
+U 1 1 5E71825B
+P 6450 4250
+AR Path="/5E5F55D4/5E71825B" Ref="#PWR?"  Part="1"
+AR Path="/5E6F1BD7/5E71825B" Ref="#PWR?"  Part="1"
+F 0 "#PWR?" H 6450 4000 50  0001 C CNN
+F 1 "GND" H 6455 4077 50  0000 C CNN
+F 2 "" H 6450 4250 50  0001 C CNN
+F 3 "" H 6450 4250 50  0001 C CNN
+	1    6450 4250
+	1    0    0    -1
+$EndComp
+Wire Wire Line
+	6400 4100 6550 4100
+Wire Wire Line
+	5800 2700 6550 2700
+Connection ~ 5800 2700
+Wire Wire Line
+	6550 2700 6550 4100
+Connection ~ 6550 2700
+Wire Wire Line
+	6550 2700 6800 2700
 $EndSCHEMATC
