File: Motors & Motors Drivers.sch (KiCad schematic (older format))
At the start: 4 parts, among them J2 Conn_01x02, J3 Conn_01x02, U4 DRV8835

Commit message: Changes in graphics, added capacitors, changes in xshut
Parts:
- added C23: 0.1uF, Capacitor_SMD:C_0402_1005Metric, symbol Device:C_Small
Connections:
- net +6V: now also C23.1
- net GND: now also C23.2
Changed lines of the file:
@@
 	1    0    0    1
 $EndComp
+$Comp
+L Device:C_Small C23
+U 1 1 5E6E22A6
+P 6400 2900
+F 0 "C23" H 6492 2946 50  0000 L CNN
+F 1 "0.1uF" H 6492 2855 50  0000 L CNN
+F 2 "Capacitor_SMD:C_0402_1005Metric" H 6400 2900 50  0001 C CNN
+F 3 "~" H 6400 2900 50  0001 C CNN
+	1    6400 2900
+	0    -1   -1   0
+$EndComp
+$Comp
+L power:GND #PWR0227
+U 1 1 5E6E2928
+P 6500 2900
+F 0 "#PWR0227" H 6500 2650 50  0001 C CNN
+F 1 "GND" V 6500 2700 50  0000 C CNN
+F 2 "" H 6500 2900 50  0001 C CNN
+F 3 "" H 6500 2900 50  0001 C CNN
+	1    6500 2900
+	0    -1   -1   0
+$EndComp
+Wire Wire Line
+	6300 2900 6200 2900
+Connection ~ 6200 2900
 $EndSCHEMATC
