File: Motors & Motors Drivers.sch (KiCad schematic (older format))
At the start: 5 parts, among them J2 Conn_01x02, J3 Conn_01x02, U4 DRV8835

Commit message: NXP version
Parts:
- removed C23, C9: 0.1uF, Capacitor_SMD:C_0402_1005Metric, symbol Device:C_Small
- removed U4: DRV8835, Package_SON:WSON-12-1EP_3x2mm_P0.5mm_EP1x2.65, symbol drv8835:DRV8835
- added U4, U7: DRV8838, Package_SON:WSON-8-1EP_2x2mm_P0.5mm_EP0.9x1.6mm, symbol Driver_Motor:DRV8838
Connections:
- net +3V3: now also U4.8 (VCC), U7.8 (VCC)
- net +6V: now also U4.1 (VM), U7.1 (VM)
- net DRV8835_DIR_A: now also U4.6 (PH)
- net DRV8835_DIR_B: now also U7.6 (PH)
- net DRV8835_EN: now also U4.7 (~SLEEP), U7.7 (~SLEEP)
- net DRV8835_PWM_A: now also U4.5 (EN)
- net DRV8835_PWM_B: now also U7.5 (EN)
- net GND: now also U4.4 (GND), U4.9 (GND), U7.4 (GND), U7.9 (GND)
- net at J2.2 (Pin_2): now also U4.2 (OUT1)
- net at J2.1 (Pin_1): now also U4.3 (OUT2)
- net at J3.2 (Pin_2): now also U7.3 (OUT2)
- net at J3.1 (Pin_1): now also U7.2 (OUT1)
Other:
- moved on the sheet: J2, J3
Changed lines of the file:
@@
 $EndDescr
-$Comp
-L drv8835:DRV8835 U4
-U 1 1 5E6F8C5C
-P 5800 3450
-F 0 "U4" H 5800 4250 50  0000 C CNN
-F 1 "DRV8835" H 5900 4150 50  0000 C CNN
-F 2 "Package_SON:WSON-12-1EP_3x2mm_P0.5mm_EP1x2.65" H 5650 3100 50  0001 C CNN
-F 3 "http://www.ti.com/lit/ds/symlink/drv8835.pdf" H 5800 3450 50  0001 C CNN
-	1    5800 3450
-	1    0    0    -1
-$EndComp
-$Comp
-L power:+3V3 #PWR0115
-U 1 1 5E6F95EF
-P 5350 2350
-F 0 "#PWR0115" H 5350 2200 50  0001 C CNN
-F 1 "+3V3" H 5365 2523 50  0000 C CNN
-F 2 "" H 5350 2350 50  0001 C CNN
-F 3 "" H 5350 2350 50  0001 C CNN
-	1    5350 2350
-	1    0    0    -1
-$EndComp
-$Comp
-L Device:C_Small C9
-U 1 1 5E6F9D49
-P 5350 2450
-F 0 "C9" H 5442 2496 50  0000 L CNN
-F 1 "0.1uF" H 5442 2405 50  0000 L CNN
-F 2 "Capacitor_SMD:C_0402_1005Metric" H 5350 2450 50  0001 C CNN
-F 3 "~" H 5350 2450 50  0001 C CNN
-	1    5350 2450
-	1    0    0    -1
-$EndComp
-$Comp
-L power:GND #PWR0116
-U 1 1 5E6FA2C1
-P 5350 2550
-F 0 "#PWR0116" H 5350 2300 50  0001 C CNN
-F 1 "GND" H 5355 2377 50  0000 C CNN
-F 2 "" H 5350 2550 50  0001 C CNN
-F 3 "" H 5350 2550 50  0001 C CNN
-	1    5350 2550
-	1    0    0    -1
-$EndComp
-Wire Wire Line
-	5700 2700 5700 2350
-Wire Wire Line
-	5700 2350 5350 2350
-Connection ~ 5350 2350
-$Comp
-L power:GND #PWR0117
-U 1 1 5E6FBAD5
-P 5700 3850
-F 0 "#PWR0117" H 5700 3600 50  0001 C CNN
-F 1 "GND" H 5705 3677 50  0000 C CNN
-F 2 "" H 5700 3850 50  0001 C CNN
-F 3 "" H 5700 3850 50  0001 C CNN
-	1    5700 3850
-	1    0    0    -1
-$EndComp
-$Comp
-L power:GND #PWR0118
-U 1 1 5E6FBECB
-P 6200 3650
-F 0 "#PWR0118" H 6200 3400 50  0001 C CNN
-F 1 "GND" H 6205 3477 50  0000 C CNN
-F 2 "" H 6200 3650 50  0001 C CNN
-F 3 "" H 6200 3650 50  0001 C CNN
-	1    6200 3650
-	1    0    0    -1
-$EndComp
-$Comp
-L power:+6V #PWR0119
-U 1 1 5E6FE882
-P 6250 2750
-F 0 "#PWR0119" H 6250 2600 50  0001 C CNN
-F 1 "+6V" H 6265 2923 50  0000 C CNN
-F 2 "" H 6250 2750 50  0001 C CNN
-F 3 "" H 6250 2750 50  0001 C CNN
-	1    6250 2750
-	1    0    0    -1
-$EndComp
-Text HLabel 5200 2900 0    50   Input ~ 0
-DRV8835_EN
-Text HLabel 5200 3100 0    50   Input ~ 0
-DRV8835_DIR_A
-Text HLabel 5200 3200 0    50   Input ~ 0
-DRV8835_PWM_A
-Text HLabel 5200 3400 0    50   Input ~ 0
-DRV8835_DIR_B
-Text HLabel 5200 3500 0    50   Input ~ 0
-DRV8835_PWM_B
 $Comp
 L Connector_Generic:Conn_01x02 J2
 U 1 1 5E700310
-P 6400 3200
-F 0 "J2" H 6480 3192 50  0000 L CNN
-F 1 "Conn_01x02" H 6480 3101 50  0000 L CNN
-F 2 "Connector_PinHeader_1.00mm:PinHeader_1x02_P1.00mm_Vertical" H 6400 3200 50  0001 C CNN
-F 3 "~" H 6400 3200 50  0001 C CNN
-	1    6400 3200
+P 5700 2950
+F 0 "J2" H 5780 2942 50  0000 L CNN
+F 1 "Conn_01x02" H 5780 2851 50  0000 L CNN
+F 2 "Connector_PinHeader_1.00mm:PinHeader_1x02_P1.00mm_Vertical" H 5700 2950 50  0001 C CNN
+F 3 "~" H 5700 2950 50  0001 C CNN
+	1    5700 2950
 	1    0    0    1
 $EndComp
@@
 L Connector_Generic:Conn_01x02 J3
 U 1 1 5E70076C
-P 6400 3500
-F 0 "J3" H 6480 3492 50  0000 L CNN
-F 1 "Conn_01x02" H 6480 3401 50  0000 L CNN
-F 2 "Connector_PinHeader_1.00mm:PinHeader_1x02_P1.00mm_Vertical" H 6400 3500 50  0001 C CNN
-F 3 "~" H 6400 3500 50  0001 C CNN
-	1    6400 3500
-	1    0    0    1
+P 5700 4500
+F 0 "J3" H 5780 4492 50  0000 L CNN
+F 1 "Conn_01x02" H 5780 4401 50  0000 L CNN
+F 2 "Connector_PinHeader_1.00mm:PinHeader_1x02_P1.00mm_Vertical" H 5700 4500 50  0001 C CNN
+F 3 "~" H 5700 4500 50  0001 C CNN
+	1    5700 4500
+	1    0    0    -1
 $EndComp
 $Comp
-L Device:C_Small C23
-U 1 1 5E6E22A6
-P 6400 2900
-F 0 "C23" H 6492 2946 50  0000 L CNN
-F 1 "0.1uF" H 6492 2855 50  0000 L CNN
-F 2 "Capacitor_SMD:C_0402_1005Metric" H 6400 2900 50  0001 C CNN
-F 3 "~" H 6400 2900 50  0001 C CNN
-	1    6400 2900
-	0    -1   -1   0
+L Driver_Motor:DRV8838 U4
+U 1 1 6014A38B
+P 5000 2900
+F 0 "U4" H 5150 3450 50  0000 C CNN
+F 1 "DRV8838" H 5250 3350 50  0000 C CNN
+F 2 "Package_SON:WSON-8-1EP_2x2mm_P0.5mm_EP0.9x1.6mm" H 5000 2050 50  0001 C CNN
+F 3 "http://www.ti.com/lit/ds/symlink/drv8837.pdf" H 5000 2900 50  0001 C CNN
+	1    5000 2900
+	1    0    0    -1
+$EndComp
+Wire Wire Line
+	5400 2600 5500 2600
+Wire Wire Line
+	5400 3200 5500 3200
+Text HLabel 4550 2800 0    50   Input ~ 0
+DRV8835_EN
+Wire Wire Line
+	4550 2800 4600 2800
+Text HLabel 4550 3000 0    50   Input ~ 0
+DRV8835_PWM_A
+Text HLabel 4550 2900 0    50   Input ~ 0
+DRV8835_DIR_A
+Wire Wire Line
+	4600 2900 4550 2900
+Wire Wire Line
+	4600 3000 4550 3000
+$Comp
+L power:+6V #PWR0115
+U 1 1 6014FD95
+P 5050 2300
+F 0 "#PWR0115" H 5050 2150 50  0001 C CNN
+F 1 "+6V" H 5065 2473 50  0000 C CNN
+F 2 "" H 5050 2300 50  0001 C CNN
+F 3 "" H 5050 2300 50  0001 C CNN
+	1    5050 2300
+	1    0    0    -1
+$EndComp
+Wire Wire Line
+	5000 2350 5000 2400
+$Comp
+L power:+3V3 #PWR0116
+U 1 1 60150BED
+P 4850 2300
+F 0 "#PWR0116" H 4850 2150 50  0001 C CNN
+F 1 "+3V3" H 4865 2473 50  0000 C CNN
+F 2 "" H 4850 2300 50  0001 C CNN
+F 3 "" H 4850 2300 50  0001 C CNN
+	1    4850 2300
+	1    0    0    -1
+$EndComp
+Wire Wire Line
+	5050 2300 5050 2350
+Wire Wire Line
+	5050 2350 5000 2350
+Wire Wire Line
+	4850 2300 4850 2350
+Wire Wire Line
+	4850 2350 4900 2350
+Wire Wire Line
+	4900 2350 4900 2400
+$Comp
+L power:GND #PWR0117
+U 1 1 60154D71
+P 5000 3400
+F 0 "#PWR0117" H 5000 3150 50  0001 C CNN
+F 1 "GND" H 5005 3227 50  0000 C CNN
+F 2 "" H 5000 3400 50  0001 C CNN
+F 3 "" H 5000 3400 50  0001 C CNN
+	1    5000 3400
+	1    0    0    -1
 $EndComp
 $Comp
-L power:GND #PWR0227
-U 1 1 5E6E2928
-P 6500 2900
-F 0 "#PWR0227" H 6500 2650 50  0001 C CNN
-F 1 "GND" V 6500 2700 50  0000 C CNN
-F 2 "" H 6500 2900 50  0001 C CNN
-F 3 "" H 6500 2900 50  0001 C CNN
-	1    6500 2900
-	0    -1   -1   0
+L Driver_Motor:DRV8838 U7
+U 1 1 60157DB6
+P 5000 4550
+F 0 "U7" H 5150 5100 50  0000 C CNN
+F 1 "DRV8838" H 5250 5000 50  0000 C CNN
+F 2 "Package_SON:WSON-8-1EP_2x2mm_P0.5mm_EP0.9x1.6mm" H 5000 3700 50  0001 C CNN
+F 3 "http://www.ti.com/lit/ds/symlink/drv8837.pdf" H 5000 4550 50  0001 C CNN
+	1    5000 4550
+	1    0    0    -1
 $EndComp
 Wire Wire Line
-	6300 2900 6250 2900
+	5400 4250 5500 4250
 Wire Wire Line
-	6250 2750 6250 2900
-Connection ~ 6250 2900
+	5400 4850 5500 4850
+Text HLabel 4550 4450 0    50   Input ~ 0
+DRV8835_EN
 Wire Wire Line
-	6250 2900 6200 2900
+	4550 4450 4600 4450
+Text HLabel 4550 4650 0    50   Input ~ 0
+DRV8835_PWM_B
+Text HLabel 4550 4550 0    50   Input ~ 0
+DRV8835_DIR_B
+Wire Wire Line
+	4600 4550 4550 4550
+Wire Wire Line
+	4600 4650 4550 4650
+$Comp
+L power:+6V #PWR0118
+U 1 1 60157DCC
+P 5050 3950
+F 0 "#PWR0118" H 5050 3800 50  0001 C CNN
+F 1 "+6V" H 5065 4123 50  0000 C CNN
+F 2 "" H 5050 3950 50  0001 C CNN
+F 3 "" H 5050 3950 50  0001 C CNN
+	1    5050 3950
+	1    0    0    -1
+$EndComp
+Wire Wire Line
+	5000 4000 5000 4050
+$Comp
+L power:+3V3 #PWR0119
+U 1 1 60157DD3
+P 4850 3950
+F 0 "#PWR0119" H 4850 3800 50  0001 C CNN
+F 1 "+3V3" H 4865 4123 50  0000 C CNN
+F 2 "" H 4850 3950 50  0001 C CNN
+F 3 "" H 4850 3950 50  0001 C CNN
+	1    4850 3950
+	1    0    0    -1
+$EndComp
+Wire Wire Line
+	5050 3950 5050 4000
+Wire Wire Line
+	5050 4000 5000 4000
+Wire Wire Line
+	4850 3950 4850 4000
+Wire Wire Line
+	4850 4000 4900 4000
+Wire Wire Line
+	4900 4000 4900 4050
+$Comp
+L power:GND #PWR0160
+U 1 1 60157DDE
+P 5000 5050
+F 0 "#PWR0160" H 5000 4800 50  0001 C CNN
+F 1 "GND" H 5005 4877 50  0000 C CNN
+F 2 "" H 5000 5050 50  0001 C CNN
+F 3 "" H 5000 5050 50  0001 C CNN
+	1    5000 5050
+	1    0    0    -1
+$EndComp
+Wire Wire Line
+	5500 2600 5500 2850
+Wire Wire Line
+	5500 2950 5500 3200
+Wire Wire Line
+	5500 4250 5500 4500
+Wire Wire Line
+	5500 4600 5500 4850
 $EndSCHEMATC
