File: WiFi.sch (KiCad schematic (older format))
At the start: 17 parts, among them J4 USB_B_Micro, J5 ESP_01, Q2 BC847, Q3 BC847, U8 CP2102N-A01-GQFN28, U9 TS5A3167DBVR

Commit message: Usunięto rezystor przy buzzerze, poprawiono połączenia do WS2812B
Parts:
- J4: symbol Connector:USB_B_Micro -> synermycha-electronics-rescue:USB_B_Micro-Connector
Changed lines of the file:
@@
 ESP_TX
 $Comp
-L Connector:USB_B_Micro J4
+L synermycha-electronics-rescue:USB_B_Micro-Connector J4
 U 1 1 5E701B58
 P 2850 4200
 AR Path="/5E5F55AD/5E701B58" Ref="J4"  Part="1"
 AR Path="/5E79B5DD/5E701B58" Ref="J?"  Part="1"
+AR Path="/5E701B58" Ref="J4"  Part="1"
 F 0 "J4" H 2907 4667 50  0000 C CNN
 F 1 "USB_B_Micro" H 2907 4576 50  0000 C CNN
