File: TestPoints.sch (KiCad schematic (older format))
At the start: 9 parts

Commit message: Dodano projekt stacji dokującej. Poprawki ścieżek i shcematu
Parts:
- added TP10, TP11, TP12: TestPoint, TestPoint:TestPoint_Pad_D1.5mm, symbol Connector:TestPoint
Connections:
- new net D+: TP11.1
- new net D-: TP12.1
- new net ~RESET: TP10.1
Changed lines of the file:
@@
 $Descr A4 11693 8268
 encoding utf-8
-Sheet 11 12
+Sheet 10 12
 Title ""
 Date ""
@@
 Wire Wire Line
 	8100 3650 3300 3650
+$Comp
+L Connector:TestPoint TP10
+U 1 1 5F9F602F
+P 8600 2650
+F 0 "TP10" H 8658 2768 50  0000 L CNN
+F 1 "TestPoint" H 8658 2677 50  0000 L CNN
+F 2 "TestPoint:TestPoint_Pad_D1.5mm" H 8800 2650 50  0001 C CNN
+F 3 "~" H 8800 2650 50  0001 C CNN
+	1    8600 2650
+	1    0    0    -1
+$EndComp
+Wire Wire Line
+	8600 2650 8600 3750
+Wire Wire Line
+	8600 3750 3300 3750
+Text HLabel 3300 3750 0    50   Output ~ 0
+~RESET
+$Comp
+L Connector:TestPoint TP11
+U 1 1 5FA3CB88
+P 9100 2650
+F 0 "TP11" H 9158 2768 50  0000 L CNN
+F 1 "TestPoint" H 9158 2677 50  0000 L CNN
+F 2 "TestPoint:TestPoint_Pad_D1.5mm" H 9300 2650 50  0001 C CNN
+F 3 "~" H 9300 2650 50  0001 C CNN
+	1    9100 2650
+	1    0    0    -1
+$EndComp
+$Comp
+L Connector:TestPoint TP12
+U 1 1 5FA3CEE3
+P 9600 2650
+F 0 "TP12" H 9658 2768 50  0000 L CNN
+F 1 "TestPoint" H 9658 2677 50  0000 L CNN
+F 2 "TestPoint:TestPoint_Pad_D1.5mm" H 9800 2650 50  0001 C CNN
+F 3 "~" H 9800 2650 50  0001 C CNN
+	1    9600 2650
+	1    0    0    -1
+$EndComp
+Wire Wire Line
+	9100 2650 9100 3850
+Wire Wire Line
+	9100 3850 3300 3850
+Wire Wire Line
+	9600 2650 9600 3950
+Wire Wire Line
+	9600 3950 3300 3950
+Text HLabel 3300 3850 0    50   BiDi ~ 0
+D+
+Text HLabel 3300 3950 0    50   BiDi ~ 0
+D-
 $EndSCHEMATC

Commit message: NXP version
Parts:
- removed TP1, TP10, TP11, TP12, TP2, TP3, TP4, TP5, TP6, TP7, TP8, TP9: TestPoint, TestPoint:TestPoint_Pad_D1.5mm, symbol Connector:TestPoint
Changed lines of the file:
@@
 Comment4 ""
 $EndDescr
-$Comp
-L Connector:TestPoint TP1
-U 1 1 5FD2A106
-P 4000 2650
-F 0 "TP1" H 4058 2768 50  0000 L CNN
-F 1 "TestPoint" H 4058 2677 50  0000 L CNN
-F 2 "TestPoint:TestPoint_Pad_D1.5mm" H 4200 2650 50  0001 C CNN
-F 3 "~" H 4200 2650 50  0001 C CNN
-	1    4000 2650
-	1    0    0    -1
-$EndComp
-$Comp
-L Connector:TestPoint TP2
-U 1 1 5FD2A5A3
-P 4550 2650
-F 0 "TP2" H 4608 2768 50  0000 L CNN
-F 1 "TestPoint" H 4608 2677 50  0000 L CNN
-F 2 "TestPoint:TestPoint_Pad_D1.5mm" H 4750 2650 50  0001 C CNN
-F 3 "~" H 4750 2650 50  0001 C CNN
-	1    4550 2650
-	1    0    0    -1
-$EndComp
-$Comp
-L Connector:TestPoint TP3
-U 1 1 5FD2A842
-P 5050 2650
-F 0 "TP3" H 5108 2768 50  0000 L CNN
-F 1 "TestPoint" H 5108 2677 50  0000 L CNN
-F 2 "TestPoint:TestPoint_Pad_D1.5mm" H 5250 2650 50  0001 C CNN
-F 3 "~" H 5250 2650 50  0001 C CNN
-	1    5050 2650
-	1    0    0    -1
-$EndComp
-$Comp
-L Connector:TestPoint TP4
-U 1 1 5FD2AA05
-P 5550 2650
-F 0 "TP4" H 5608 2768 50  0000 L CNN
-F 1 "TestPoint" H 5608 2677 50  0000 L CNN
-F 2 "TestPoint:TestPoint_Pad_D1.5mm" H 5750 2650 50  0001 C CNN
-F 3 "~" H 5750 2650 50  0001 C CNN
-	1    5550 2650
-	1    0    0    -1
-$EndComp
-$Comp
-L Connector:TestPoint TP5
-U 1 1 5FD2BBA3
-P 6050 2650
-F 0 "TP5" H 6108 2768 50  0000 L CNN
-F 1 "TestPoint" H 6108 2677 50  0000 L CNN
-F 2 "TestPoint:TestPoint_Pad_D1.5mm" H 6250 2650 50  0001 C CNN
-F 3 "~" H 6250 2650 50  0001 C CNN
-	1    6050 2650
-	1    0    0    -1
-$EndComp
-$Comp
-L Connector:TestPoint TP6
-U 1 1 5FD2BBA9
-P 6600 2650
-F 0 "TP6" H 6658 2768 50  0000 L CNN
-F 1 "TestPoint" H 6658 2677 50  0000 L CNN
-F 2 "TestPoint:TestPoint_Pad_D1.5mm" H 6800 2650 50  0001 C CNN
-F 3 "~" H 6800 2650 50  0001 C CNN
-	1    6600 2650
-	1    0    0    -1
-$EndComp
-$Comp
-L Connector:TestPoint TP7
-U 1 1 5FD2BBAF
-P 7100 2650
-F 0 "TP7" H 7158 2768 50  0000 L CNN
-F 1 "TestPoint" H 7158 2677 50  0000 L CNN
-F 2 "TestPoint:TestPoint_Pad_D1.5mm" H 7300 2650 50  0001 C CNN
-F 3 "~" H 7300 2650 50  0001 C CNN
-	1    7100 2650
-	1    0    0    -1
-$EndComp
 Text HLabel 3300 2850 0    50   Output ~ 0
 SWDCLK
@@
 Wire Wire Line
 	3300 3450 7100 3450
-$Comp
-L Connector:TestPoint TP8
-U 1 1 5FE4475E
-P 7600 2650
-F 0 "TP8" H 7658 2768 50  0000 L CNN
-F 1 "TestPoint" H 7658 2677 50  0000 L CNN
-F 2 "TestPoint:TestPoint_Pad_D1.5mm" H 7800 2650 50  0001 C CNN
-F 3 "~" H 7800 2650 50  0001 C CNN
-	1    7600 2650
-	1    0    0    -1
-$EndComp
-$Comp
-L Connector:TestPoint TP9
-U 1 1 5FE44C0F
-P 8100 2650
-F 0 "TP9" H 8158 2768 50  0000 L CNN
-F 1 "TestPoint" H 8158 2677 50  0000 L CNN
-F 2 "TestPoint:TestPoint_Pad_D1.5mm" H 8300 2650 50  0001 C CNN
-F 3 "~" H 8300 2650 50  0001 C CNN
-	1    8100 2650
-	1    0    0    -1
-$EndComp
 Text HLabel 3300 3550 0    50   BiDi ~ 0
 CC1
@@
 Wire Wire Line
 	8100 3650 3300 3650
-$Comp
-L Connector:TestPoint TP10
-U 1 1 5F9F602F
-P 8600 2650
-F 0 "TP10" H 8658 2768 50  0000 L CNN
-F 1 "TestPoint" H 8658 2677 50  0000 L CNN
-F 2 "TestPoint:TestPoint_Pad_D1.5mm" H 8800 2650 50  0001 C CNN
-F 3 "~" H 8800 2650 50  0001 C CNN
-	1    8600 2650
-	1    0    0    -1
-$EndComp
 Wire Wire Line
 	8600 2650 8600 3750
@@
 Text HLabel 3300 3750 0    50   Output ~ 0
 ~RESET
-$Comp
-L Connector:TestPoint TP11
-U 1 1 5FA3CB88
-P 9100 2650
-F 0 "TP11" H 9158 2768 50  0000 L CNN
-F 1 "TestPoint" H 9158 2677 50  0000 L CNN
-F 2 "TestPoint:TestPoint_Pad_D1.5mm" H 9300 2650 50  0001 C CNN
-F 3 "~" H 9300 2650 50  0001 C CNN
-	1    9100 2650
-	1    0    0    -1
-$EndComp
-$Comp
-L Connector:TestPoint TP12
-U 1 1 5FA3CEE3
-P 9600 2650
-F 0 "TP12" H 9658 2768 50  0000 L CNN
-F 1 "TestPoint" H 9658 2677 50  0000 L CNN
-F 2 "TestPoint:TestPoint_Pad_D1.5mm" H 9800 2650 50  0001 C CNN
-F 3 "~" H 9800 2650 50  0001 C CNN
-	1    9600 2650
-	1    0    0    -1
-$EndComp
 Wire Wire Line
 	9100 2650 9100 3850
