File: LED & Oled & Buzzer.sch (KiCad schematic (older format))
At the start: 17 parts, among them J6 A1250WV-S-4P, Q4 BC847

Commit message: NXP version
Parts:
- removed D2, D3, D4, D5: RED, 5mA, LED_SMD:LED_0402_1005Metric, symbol Device:LED_Small
- removed D6: RED, LED_SMD:LED_0402_1005Metric, symbol Device:LED_Small
- removed R22, R23, R24, R25, R26: 270, Resistor_SMD:R_0402_1005Metric, symbol Device:R_Small
Changed lines of the file:
@@
 Text HLabel 3100 4350 0    50   Input ~ 0
 BUZZER
-$Comp
-L Device:LED_Small D2
-U 1 1 5E6BFB7A
-P 6600 1700
-F 0 "D2" V 6554 1798 50  0000 L CNN
-F 1 "RED, 5mA" V 6645 1798 50  0000 L CNN
-F 2 "LED_SMD:LED_0402_1005Metric" V 6600 1700 50  0001 C CNN
-F 3 "~" V 6600 1700 50  0001 C CNN
-	1    6600 1700
-	0    1    1    0
-$EndComp
-$Comp
-L Device:R_Small R22
-U 1 1 5E6C3B93
-P 6600 1500
-F 0 "R22" H 6541 1454 50  0000 R CNN
-F 1 "270" H 6541 1545 50  0000 R CNN
-F 2 "Resistor_SMD:R_0402_1005Metric" H 6600 1500 50  0001 C CNN
-F 3 "~" H 6600 1500 50  0001 C CNN
-	1    6600 1500
-	-1   0    0    1
-$EndComp
-Wire Wire Line
-	6600 1800 6600 1850
-Wire Wire Line
-	6600 1850 6400 1850
-$Comp
-L Device:LED_Small D3
-U 1 1 5E6C6876
-P 7000 1700
-F 0 "D3" V 6954 1798 50  0000 L CNN
-F 1 "RED, 5mA" V 7045 1798 50  0000 L CNN
-F 2 "LED_SMD:LED_0402_1005Metric" V 7000 1700 50  0001 C CNN
-F 3 "~" V 7000 1700 50  0001 C CNN
-	1    7000 1700
-	0    1    1    0
-$EndComp
-$Comp
-L Device:R_Small R23
-U 1 1 5E6C6882
-P 7000 1500
-F 0 "R23" H 6941 1454 50  0000 R CNN
-F 1 "270" H 6941 1545 50  0000 R CNN
-F 2 "Resistor_SMD:R_0402_1005Metric" H 7000 1500 50  0001 C CNN
-F 3 "~" H 7000 1500 50  0001 C CNN
-	1    7000 1500
-	-1   0    0    1
-$EndComp
-$Comp
-L Device:LED_Small D4
-U 1 1 5E6C73DF
-P 7350 1700
-F 0 "D4" V 7304 1798 50  0000 L CNN
-F 1 "RED, 5mA" V 7395 1798 50  0000 L CNN
-F 2 "LED_SMD:LED_0402_1005Metric" V 7350 1700 50  0001 C CNN
-F 3 "~" V 7350 1700 50  0001 C CNN
-	1    7350 1700
-	0    1    1    0
-$EndComp
-$Comp
-L Device:R_Small R24
-U 1 1 5E6C73EB
-P 7350 1500
-F 0 "R24" H 7291 1454 50  0000 R CNN
-F 1 "270" H 7291 1545 50  0000 R CNN
-F 2 "Resistor_SMD:R_0402_1005Metric" H 7350 1500 50  0001 C CNN
-F 3 "~" H 7350 1500 50  0001 C CNN
-	1    7350 1500
-	-1   0    0    1
-$EndComp
-$Comp
-L Device:LED_Small D5
-U 1 1 5E6C7B05
-P 7700 1700
-F 0 "D5" V 7654 1798 50  0000 L CNN
-F 1 "RED, 5mA" V 7745 1798 50  0000 L CNN
-F 2 "LED_SMD:LED_0402_1005Metric" V 7700 1700 50  0001 C CNN
-F 3 "~" V 7700 1700 50  0001 C CNN
-	1    7700 1700
-	0    1    1    0
-$EndComp
-$Comp
-L Device:R_Small R25
-U 1 1 5E6C7B11
-P 7700 1500
-F 0 "R25" H 7641 1454 50  0000 R CNN
-F 1 "270" H 7641 1545 50  0000 R CNN
-F 2 "Resistor_SMD:R_0402_1005Metric" H 7700 1500 50  0001 C CNN
-F 3 "~" H 7700 1500 50  0001 C CNN
-	1    7700 1500
-	-1   0    0    1
-$EndComp
-$Comp
-L Device:R_Small R26
-U 1 1 5E6C8421
-P 8050 1500
-F 0 "R26" H 7991 1454 50  0000 R CNN
-F 1 "270" H 7991 1545 50  0000 R CNN
-F 2 "Resistor_SMD:R_0402_1005Metric" H 8050 1500 50  0001 C CNN
-F 3 "~" H 8050 1500 50  0001 C CNN
-	1    8050 1500
-	-1   0    0    1
-$EndComp
-Wire Wire Line
-	7000 1800 7000 1950
-Wire Wire Line
-	7000 1950 6400 1950
-Wire Wire Line
-	7350 1800 7350 2050
-Wire Wire Line
-	7350 2050 6400 2050
-Wire Wire Line
-	7700 1800 7700 2150
-Wire Wire Line
-	7700 2150 6400 2150
-Wire Wire Line
-	8050 1800 8050 2250
-Wire Wire Line
-	8050 2250 6400 2250
-Text HLabel 6400 1850 0    50   Input ~ 0
-~LED_1
-Text HLabel 6400 1950 0    50   Input ~ 0
-~LED_2
-Text HLabel 6400 2050 0    50   Input ~ 0
-~LED_3
-Text HLabel 6400 2150 0    50   Input ~ 0
-~LED_4
-Text HLabel 6400 2250 0    50   Input ~ 0
-~LED_5
 Wire Wire Line
 	3600 3700 3600 3650
@@
 	3600 3900 3500 3900
 Connection ~ 3600 3900
-$Comp
-L Device:LED_Small D6
-U 1 1 5E6C8415
-P 8050 1700
-F 0 "D6" V 8004 1798 50  0000 L CNN
-F 1 "RED" V 8095 1798 50  0000 L CNN
-F 2 "LED_SMD:LED_0402_1005Metric" V 8050 1700 50  0001 C CNN
-F 3 "~" V 8050 1700 50  0001 C CNN
-	1    8050 1700
-	0    1    1    0
-$EndComp
 $Comp
 L Device:R_Small R27
@@
 	8900 1800 8900 2600
 $Comp
-L power:GND #PWR0160
-U 1 1 5F93DEEE
-P 6600 1400
-F 0 "#PWR0160" H 6600 1150 50  0001 C CNN
-F 1 "GND" H 6605 1227 50  0000 C CNN
-F 2 "" H 6600 1400 50  0001 C CNN
-F 3 "" H 6600 1400 50  0001 C CNN
-	1    6600 1400
-	-1   0    0    1
-$EndComp
-$Comp
-L power:GND #PWR0161
-U 1 1 5F93E3AF
-P 7000 1400
-F 0 "#PWR0161" H 7000 1150 50  0001 C CNN
-F 1 "GND" H 7005 1227 50  0000 C CNN
-F 2 "" H 7000 1400 50  0001 C CNN
-F 3 "" H 7000 1400 50  0001 C CNN
-	1    7000 1400
-	-1   0    0    1
-$EndComp
-$Comp
-L power:GND #PWR0162
-U 1 1 5F93E75E
-P 7350 1400
-F 0 "#PWR0162" H 7350 1150 50  0001 C CNN
-F 1 "GND" H 7355 1227 50  0000 C CNN
-F 2 "" H 7350 1400 50  0001 C CNN
-F 3 "" H 7350 1400 50  0001 C CNN
-	1    7350 1400
-	-1   0    0    1
-$EndComp
-$Comp
-L power:GND #PWR0163
-U 1 1 5F93EBB2
-P 7700 1400
-F 0 "#PWR0163" H 7700 1150 50  0001 C CNN
-F 1 "GND" H 7705 1227 50  0000 C CNN
-F 2 "" H 7700 1400 50  0001 C CNN
-F 3 "" H 7700 1400 50  0001 C CNN
-	1    7700 1400
-	-1   0    0    1
-$EndComp
-$Comp
-L power:GND #PWR0164
-U 1 1 5F93EF9E
-P 8050 1400
-F 0 "#PWR0164" H 8050 1150 50  0001 C CNN
-F 1 "GND" H 8055 1227 50  0000 C CNN
-F 2 "" H 8050 1400 50  0001 C CNN
-F 3 "" H 8050 1400 50  0001 C CNN
-	1    8050 1400
-	-1   0    0    1
-$EndComp
-$Comp
 L power:GND #PWR0165
