File: Buttonssch.sch (KiCad schematic (older format))
At the start: 12 parts, among them SW1 DTSM32N, SW2 DTSM32N, SW3 DTSM32N, SW4 DTSM32N

Commit message: Holy $hi3t
Parts:
- added R14, R15, R5, R6: R_Small, Resistor_SMD:R_0402_1005Metric, symbol Device:R_Small
Connections:
- net GND: now also R14.2, R15.2, R5.2, R6.2; no longer SW1.1, SW2.1, SW3.1, SW4.1
- new net: R5.1, SW1.1
- new net: R6.1, SW2.1
- new net: R14.1, SW3.1
- new net: R15.1, SW4.1
Changed lines of the file:
@@
-	1    0    0    -1
-$EndComp
-$Comp
-L power:GND #PWR0122
-U 1 1 5E639B26
-P 4750 2150
-F 0 "#PWR0122" H 4750 1900 50  0001 C CNN
-F 1 "GND" H 4755 1977 50  0000 C CNN
-F 2 "" H 4750 2150 50  0001 C CNN
-F 3 "" H 4750 2150 50  0001 C CNN
-	1    4750 2150
 	1    0    0    -1
 $EndComp
@@
 L power:GND #PWR0125
 U 1 1 5E63C481
-P 4750 3150
-F 0 "#PWR0125" H 4750 2900 50  0001 C CNN
-F 1 "GND" H 4755 2977 50  0000 C CNN
-F 2 "" H 4750 3150 50  0001 C CNN
-F 3 "" H 4750 3150 50  0001 C CNN
-	1    4750 3150
+P 4550 3150
+F 0 "#PWR0125" H 4550 2900 50  0001 C CNN
+F 1 "GND" H 4555 2977 50  0000 C CNN
+F 2 "" H 4550 3150 50  0001 C CNN
+F 3 "" H 4550 3150 50  0001 C CNN
+	1    4550 3150
 	1    0    0    -1
 $EndComp
@@
 	1    0    0    -1
 $EndComp
-$Comp
-L power:GND #PWR0128
-U 1 1 5E63DF9E
-P 4750 4100
-F 0 "#PWR0128" H 4750 3850 50  0001 C CNN
-F 1 "GND" H 4755 3927 50  0000 C CNN
-F 2 "" H 4750 4100 50  0001 C CNN
-F 3 "" H 4750 4100 50  0001 C CNN
-	1    4750 4100
-	1    0    0    -1
-$EndComp
 Wire Wire Line
 	5150 4100 6200 4100
@@
 	1    0    0    -1
 $EndComp
-$Comp
-L power:GND #PWR0131
-U 1 1 5E640E19
-P 4750 5050
-F 0 "#PWR0131" H 4750 4800 50  0001 C CNN
-F 1 "GND" H 4755 4877 50  0000 C CNN
-F 2 "" H 4750 5050 50  0001 C CNN
-F 3 "" H 4750 5050 50  0001 C CNN
-	1    4750 5050
-	1    0    0    -1
-$EndComp
 Wire Wire Line
 	5150 5050 6200 5050
 Text HLabel 6200 5050 2    50   Output ~ 0
 ~BUTTON_OK
+$Comp
+L Device:R_Small R6
+U 1 1 5F8747F7
+P 4650 3150
+F 0 "R6" V 4454 3150 50  0000 C CNN
+F 1 "R_Small" V 4545 3150 50  0000 C CNN
+F 2 "Resistor_SMD:R_0402_1005Metric" H 4650 3150 50  0001 C CNN
+F 3 "~" H 4650 3150 50  0001 C CNN
+	1    4650 3150
+	0    1    1    0
+$EndComp
+$Comp
+L power:GND #PWR0122
+U 1 1 5F8779D0
+P 4550 4100
+F 0 "#PWR0122" H 4550 3850 50  0001 C CNN
+F 1 "GND" H 4555 3927 50  0000 C CNN
+F 2 "" H 4550 4100 50  0001 C CNN
+F 3 "" H 4550 4100 50  0001 C CNN
+	1    4550 4100
+	1    0    0    -1
+$EndComp
+$Comp
+L Device:R_Small R14
+U 1 1 5F8779D6
+P 4650 4100
+F 0 "R14" V 4454 4100 50  0000 C CNN
+F 1 "R_Small" V 4545 4100 50  0000 C CNN
+F 2 "Resistor_SMD:R_0402_1005Metric" H 4650 4100 50  0001 C CNN
+F 3 "~" H 4650 4100 50  0001 C CNN
+	1    4650 4100
+	0    1    1    0
+$EndComp
+$Comp
+L power:GND #PWR0128
+U 1 1 5F877FEA
+P 4550 5050
+F 0 "#PWR0128" H 4550 4800 50  0001 C CNN
+F 1 "GND" H 4555 4877 50  0000 C CNN
+F 2 "" H 4550 5050 50  0001 C CNN
+F 3 "" H 4550 5050 50  0001 C CNN
+	1    4550 5050
+	1    0    0    -1
+$EndComp
+$Comp
+L Device:R_Small R15
+U 1 1 5F877FF0
+P 4650 5050
+F 0 "R15" V 4454 5050 50  0000 C CNN
+F 1 "R_Small" V 4545 5050 50  0000 C CNN
+F 2 "Resistor_SMD:R_0402_1005Metric" H 4650 5050 50  0001 C CNN
+F 3 "~" H 4650 5050 50  0001 C CNN
+	1    4650 5050
+	0    1    1    0
+$EndComp
+$Comp
+L power:GND #PWR0131
+U 1 1 5F878884
+P 4550 2150
+F 0 "#PWR0131" H 4550 1900 50  0001 C CNN
+F 1 "GND" H 4555 1977 50  0000 C CNN
+F 2 "" H 4550 2150 50  0001 C CNN
+F 3 "" H 4550 2150 50  0001 C CNN
+	1    4550 2150
+	1    0    0    -1
+$EndComp
+$Comp
+L Device:R_Small R5
+U 1 1 5F87888A
+P 4650 2150
+F 0 "R5" V 4454 2150 50  0000 C CNN
+F 1 "R_Small" V 4545 2150 50  0000 C CNN
+F 2 "Resistor_SMD:R_0402_1005Metric" H 4650 2150 50  0001 C CNN
+F 3 "~" H 4650 2150 50  0001 C CNN
+	1    4650 2150
+	0    1    1    0
+$EndComp
 $EndSCHEMATC

Commit message: NXP version
Parts:
- removed C11, C12, C13: 1uF, Capacitor_SMD:C_0402_1005Metric, symbol Device:C_Small
- removed R10, R8, R9: 10K, Resistor_SMD:R_0402_1005Metric, symbol Device:R_Small
- removed R14, R15: R_Small, Resistor_SMD:R_0402_1005Metric, symbol Device:R_Small
- removed SW1, SW2, SW3, SW4: DTSM32N, Button_Switch_SMD:SW_SPST_B3U-1000P, symbol Switch:SW_Push
- added RN1: R_Pack05, Resistor_SMD:R_Array_Convex_5x0603, symbol Device:R_Pack05
- added S1: SKRPACE010, footprints:SW_SKRPACE010, symbol SKRPACE010:SKRPACE010
- added S2: SKRHABE010, footprints:SKRHABE010, symbol SKRHABE010:SKRHABE010
Connections:
- net GND: now also R6.1, RN1.1 (R1.1), RN1.2 (R2.1), RN1.3 (R3.1), RN1.4 (R4.1), RN1.5 (R5.1); no longer R6.2
- net ~BUTTON_DOWN: now also RN1.9 (R2.2), S2.6 (D)
- net ~BUTTON_OK: now also RN1.7 (R4.2), S2.2 (CENTER)
- net ~BUTTON_UP: now also RN1.10 (R1.2), S2.4 (B)
- net ~RESET: now also S1.1, S1.2
- net at R5.1: now also S1.3, S1.4
- new net: R6.2, S2.5 (COMMON)
- new net ~BUTTON_LEFT: RN1.6 (R5.2), S2.1 (A)
- new net ~BUTTON_RIGHT: RN1.8 (R3.2), S2.3 (C)
- no-connect marks 0 -> 2
Other:
- moved on the sheet: R5

Commit message: Back to STM, added level shifter for RGB
Parts:
- C10: footprint Capacitor_SMD:C_0402_1005Metric -> Capacitor_SMD:C_0201_0603Metric
Changed lines of the file:
@@
 F 0 "C10" H 5242 2296 50  0000 L CNN
 F 1 "1uF" H 5242 2205 50  0000 L CNN
-F 2 "Capacitor_SMD:C_0402_1005Metric" H 5150 2250 50  0001 C CNN
+F 2 "Capacitor_SMD:C_0201_0603Metric" H 5150 2250 50  0001 C CNN
 F 3 "~" H 5150 2250 50  0001 C CNN
 	1    5150 2250
