File: microcontroller.kicad_sch (KiCad schematic)
At the start: 40 parts

Commit message: Change naming from SOM to MCU
Connections:
- net SOM_DCDC_PSWITCH renamed MCU_DCDC_PSWITCH
- net SOM_NVCC_PLL renamed MCU_NVCC_PLL
- net SOM_ONOFF renamed MCU_ONOFF
- net SOM_PMIC_ON_REQ renamed MCU_PMIC_ON_REQ
- net SOM_PMIC_STBT_REQ renamed MCU_PMIC_STBT_REQ
- net SOM_POR_B renamed MCU_POR_B
- net SOM_VDD_HIGH_CAP renamed MCU_VDD_HIGH_CAP
- net SOM_VDD_SNVS_CAP renamed MCU_VDD_SNVS_CAP
- net SOM_VDD_USB_VCAP renamed MCU_VDD_USB_VCAP
- net SOM_WAKEUP renamed MCU_WAKEUP
Other:
- note added: "MCU GPIO"
- note added: "MCU POWER & CTRL"
- note removed: "SOM GPIO"
- note removed: "SOM POWER & CTRL"

Commit message: Annotate parts, add more buses
Parts:
- added C?: C_220n_0402, antmicro-footprints:0402-cap, symbol antmicroCapacitors0402:C_220n_0402
- added J?: USB4105-GF-A, antmicro-footprints:GCT_USB4105-GF-A, symbol antmicroUSBDVIHDMIConnectors:USB4105-GF-A
- added U?: W25Q64JVXGIM, antmicro-footprints:WSON-8-1EP_4x4mm_P0.8mm_EP2.6x3mm, symbol antmicroMemory:W25Q64JVXGIM
- gave numbers to parts that had none: 38
Connections:
- net +3V3: now also C?.1, U?.8 (VCC)
- net GND: now also C?.2, J?.A1 (GND), J?.A12 (GND), J?.B1 (GND), J?.B12 (GND), J?.S1 (SHIELD), U?.4 (GND); no longer U8.G14 (GPIO_AD_B0_05)
- net MCU_DCDC_IN: now reaches C37.1, C40.1, C45.1, FB1.2, U8.K4 (DCDC_IN_Q), U8.L1 (DCDC_IN), U8.L2 (DCDC_IN)
- net PSRAM.DATA1: now reaches U8.A2 (GPIO_EMC_27)
- net PSRAM.DATA1: now also U?.2 (DO/IO1)
- net PSRAM.DATA0: now reaches U8.B3 (GPIO_EMC_26)
- net PSRAM.DATA0: now also U?.5 (DI/IO0)
- net PSRAM.DATA2: now reaches U8.D1 (GPIO_EMC_28)
- net PSRAM.DATA2: now also U?.3 (~{WP}/IO2)
- net PSRAM.CLK: now reaches U8.D2 (GPIO_EMC_25)
- net PSRAM.CLK: now also U?.6 (CLK)
- net PSRAM.~{CS}: now reaches U8.D3 (GPIO_EMC_24)
- net PSRAM.DATA3: now reaches U8.E1 (GPIO_EMC_29)
- net PSRAM.DATA3: now also U?.7 (~{HLD}/~{RST}/IO3)
- net PSRAM.~{CS1}: now reaches U8.F1 (GPIO_EMC_22)
- net PSRAM.~{CS1}: now also U?.1 (~{CS})
- net USB1.VBUS: now reaches U8.N6 (USB_OTG1_VBUS)
- net USB1.VBUS: now also J?.A4 (VBUS), J?.A9 (VBUS), J?.B4 (VBUS), J?.B9 (VBUS)
- net FLASH_CLK renamed FLASH.CLK
- net FLASH_IO0 renamed FLASH.DATA0
- net FLASH_IO1 renamed FLASH.DATA1
- net FLASH_IO2 renamed FLASH.DATA2
- net FLASH_IO3 renamed FLASH.DATA3
- net JTAG_TCK renamed JTAG.TCK
- net JTAG_TDI renamed JTAG.TDI
- net JTAG_TDO renamed JTAG.TDO
- net JTAG_TMS renamed JTAG.TMS
- net SD_CLK renamed SD.CLK
- net SD_CMD renamed SD.CMD
- net SD_DAT0 renamed SD.DATA0
- net SD_DAT1 renamed SD.DATA1
- net SD_DAT2 renamed SD.DATA2
- net SD_DAT3 renamed SD.DATA3
- net USB_DN renamed USB1.DN
- net USB1.DN: now also J?.A7 (D-), J?.B7 (D-)
- net USB_DP renamed USB1.DP
- net USB1.DP: now also J?.A6 (D+), J?.B6 (D+)
- net ~{FLASH_CS} renamed FLASH.~{CS}
- new net BOOT_MODE1: U8.G14 (GPIO_AD_B0_05)
- no-connect marks 2 -> 6
Other:
- note added: "ADDITIONAL PSRAM, FLASH (OPTION)"
- note added: "OTG USB CONNECTOR"
- note removed: "PSRAM (OPTION)"
- moved on the sheet: C51, C52, J1, TP13, TP14, U10, U9

Commit message: Add more buses
Parts:
- gave numbers to parts that had none: 3
