File: bluetooth.kicad_sch (KiCad schematic)
At the start: 5 parts, among them Q5 BC856, U3 RN4871U-V_RM118

Commit message: Cleanup bluetooth schematic
Parts:
- removed AE1: Antenna_Chip, RF_Antenna:Johanson_2450AT18x100, symbol Device:Antenna_Chip
- removed Q5: BC856, Package_TO_SOT_SMD:SOT-23, symbol Transistor_BJT:BC856
- removed R59, R60: 10K, Resistor_SMD:R_0402_1005Metric, symbol Device:R_Small
- removed U3: RN4871U-V_RM118, eec:Microchip-RN4871U-V_RM118-0, symbol eec:RN4871U-V_RM118
Connections:
- no-connect marks 9 -> 0
