File: rgb.kicad_sch (KiCad schematic)
At the start: 10 parts

Commit message: Cleanup RGB schematic
Parts:
- removed D10, D11, D12, D13, D20, D21, D22, D7, D8, D9: WS2812B_2020, WS2812-2020:WS28122020, symbol synermycha-electronics:WS2812B_2020
Connections:
- no-connect marks 2 -> 1
Changed lines of the file:
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@@
   (junction (at 199.39 113.03) (diameter 0) (color 0 0 0 0)
   )
-  (no_connect (at 222.25 102.87))
   (no_connect (at 298.45 87.63))
   (wire (pts (xy 72.39 90.17) (xy 77.47 90.17))
@@
     (stroke (width 0) (type default) (color 0 0 0 0))
   )
-  (hierarchical_label "WS2812B_IN" (shape input) (at 69.85 102.87 180)
-    (effects (font (size 1.27 1.27)) (justify right))
-  )
   (symbol (lib_id "power:GND") (at 72.39 113.03 0) (unit 1)
     (in_bom yes) (on_board yes)
@@
     (pin "1")
   )
-  (symbol (lib_id "synermycha-electronics:WS2812B_2020") (at 77.47 102.87 0) (unit 1)
-    (in_bom yes) (on_board yes)
-    (property "Reference" "D7" (id 0) (at 80.01 96.52 0)
-      (effects (font (size 1.27 1.27)) (justify left))
-    )
-    (property "Value" "WS2812B_2020" (id 1) (at 69.85 93.98 0)
-      (effects (font (size 1.27 1.27)) (justify left))
-    )
-    (property "Footprint" "WS2812-2020:WS28122020" (id 2) (at 78.74 110.49 0)
-      (effects (font (size 1.27 1.27)) (justify left top) hide)
-    )
-    (property "Datasheet" "https://cdn-shop.adafruit.com/datasheets/WS2812B.pdf" (id 3) (at 80.01 112.395 0)
-      (effects (font (size 1.27 1.27)) (justify left top) hide)
-    )
-    (pin "1")
-    (pin "2")
-    (pin "3")
-    (pin "4")
-  )
-  (symbol (lib_id "synermycha-electronics:WS2812B_2020") (at 92.71 102.87 0) (unit 1)
-    (in_bom yes) (on_board yes)
-    (property "Reference" "D8" (id 0) (at 95.25 96.52 0)
-      (effects (font (size 1.27 1.27)) (justify left))
-    )
-    (property "Value" "WS2812B_2020" (id 1) (at 85.09 93.98 0)
-      (effects (font (size 1.27 1.27)) (justify left))
-    )
-    (property "Footprint" "WS2812-2020:WS28122020" (id 2) (at 93.98 110.49 0)
-      (effects (font (size 1.27 1.27)) (justify left top) hide)
-    )
-    (property "Datasheet" "https://cdn-shop.adafruit.com/datasheets/WS2812B.pdf" (id 3) (at 95.25 112.395 0)
-      (effects (font (size 1.27 1.27)) (justify left top) hide)
-    )
-    (pin "1")
-    (pin "2")
-    (pin "3")
-    (pin "4")
-  )
-  (symbol (lib_id "synermycha-electronics:WS2812B_2020") (at 107.95 102.87 0) (unit 1)
-    (in_bom yes) (on_board yes)
-    (property "Reference" "D9" (id 0) (at 110.49 96.52 0)
-      (effects (font (size 1.27 1.27)) (justify left))
-    )
-    (property "Value" "WS2812B_2020" (id 1) (at 100.33 93.98 0)
-      (effects (font (size 1.27 1.27)) (justify left))
-    )
-    (property "Footprint" "WS2812-2020:WS28122020" (id 2) (at 109.22 110.49 0)
-      (effects (font (size 1.27 1.27)) (justify left top) hide)
-    )
-    (property "Datasheet" "https://cdn-shop.adafruit.com/datasheets/WS2812B.pdf" (id 3) (at 110.49 112.395 0)
-      (effects (font (size 1.27 1.27)) (justify left top) hide)
-    )
-    (pin "1")
-    (pin "2")
-    (pin "3")
-    (pin "4")
-  )
-  (symbol (lib_id "synermycha-electronics:WS2812B_2020") (at 138.43 102.87 0) (unit 1)
-    (in_bom yes) (on_board yes)
-    (property "Reference" "D10" (id 0) (at 140.97 96.52 0)
-      (effects (font (size 1.27 1.27)) (justify left))
-    )
-    (property "Value" "WS2812B_2020" (id 1) (at 130.81 93.98 0)
-      (effects (font (size 1.27 1.27)) (justify left))
-    )
-    (property "Footprint" "WS2812-2020:WS28122020" (id 2) (at 139.7 110.49 0)
-      (effects (font (size 1.27 1.27)) (justify left top) hide)
-    )
-    (property "Datasheet" "https://cdn-shop.adafruit.com/datasheets/WS2812B.pdf" (id 3) (at 140.97 112.395 0)
-      (effects (font (size 1.27 1.27)) (justify left top) hide)
-    )
-    (pin "1")
-    (pin "2")
-    (pin "3")
-    (pin "4")
-  )
-  (symbol (lib_id "synermycha-electronics:WS2812B_2020") (at 168.91 102.87 0) (unit 1)
-    (in_bom yes) (on_board yes)
-    (property "Reference" "D11" (id 0) (at 171.45 96.52 0)
-      (effects (font (size 1.27 1.27)) (justify left))
-    )
-    (property "Value" "WS2812B_2020" (id 1) (at 161.29 93.98 0)
-      (effects (font (size 1.27 1.27)) (justify left))
-    )
-    (property "Footprint" "WS2812-2020:WS28122020" (id 2) (at 170.18 110.49 0)
-      (effects (font (size 1.27 1.27)) (justify left top) hide)
-    )
-    (property "Datasheet" "https://cdn-shop.adafruit.com/datasheets/WS2812B.pdf" (id 3) (at 171.45 112.395 0)
-      (effects (font (size 1.27 1.27)) (justify left top) hide)
-    )
-    (pin "1")
-    (pin "2")
-    (pin "3")
-    (pin "4")
-  )
-  (symbol (lib_id "synermycha-electronics:WS2812B_2020") (at 184.15 102.87 0) (unit 1)
-    (in_bom yes) (on_board yes)
-    (property "Reference" "D12" (id 0) (at 186.69 96.52 0)
-      (effects (font (size 1.27 1.27)) (justify left))
-    )
-    (property "Value" "WS2812B_2020" (id 1) (at 176.53 93.98 0)
-      (effects (font (size 1.27 1.27)) (justify left))
-    )
-    (property "Footprint" "WS2812-2020:WS28122020" (id 2) (at 185.42 110.49 0)
-      (effects (font (size 1.27 1.27)) (justify left top) hide)
-    )
-    (property "Datasheet" "https://cdn-shop.adafruit.com/datasheets/WS2812B.pdf" (id 3) (at 186.69 112.395 0)
-      (effects (font (size 1.27 1.27)) (justify left top) hide)
-    )
-    (pin "1")
-    (pin "2")
-    (pin "3")
-    (pin "4")
-  )
-  (symbol (lib_id "synermycha-electronics:WS2812B_2020") (at 199.39 102.87 0) (unit 1)
-    (in_bom yes) (on_board yes)
-    (property "Reference" "D13" (id 0) (at 201.93 96.52 0)
-      (effects (font (size 1.27 1.27)) (justify left))
-    )
-    (property "Value" "WS2812B_2020" (id 1) (at 191.77 93.98 0)
-      (effects (font (size 1.27 1.27)) (justify left))
-    )
-    (property "Footprint" "WS2812-2020:WS28122020" (id 2) (at 200.66 110.49 0)
-      (effects (font (size 1.27 1.27)) (justify left top) hide)
-    )
-    (property "Datasheet" "https://cdn-shop.adafruit.com/datasheets/WS2812B.pdf" (id 3) (at 201.93 112.395 0)
-      (effects (font (size 1.27 1.27)) (justify left top) hide)
-    )
-    (pin "1")
-    (pin "2")
-    (pin "3")
-    (pin "4")
-  )
-  (symbol (lib_id "synermycha-electronics:WS2812B_2020") (at 153.67 102.87 0) (unit 1)
-    (in_bom yes) (on_board yes)
-    (property "Reference" "D21" (id 0) (at 156.21 96.52 0)
-      (effects (font (size 1.27 1.27)) (justify left))
-    )
-    (property "Value" "WS2812B_2020" (id 1) (at 146.05 93.98 0)
-      (effects (font (size 1.27 1.27)) (justify left))
-    )
-    (property "Footprint" "WS2812-2020:WS28122020" (id 2) (at 154.94 110.49 0)
-      (effects (font (size 1.27 1.27)) (justify left top) hide)
-    )
-    (property "Datasheet" "https://cdn-shop.adafruit.com/datasheets/WS2812B.pdf" (id 3) (at 156.21 112.395 0)
-      (effects (font (size 1.27 1.27)) (justify left top) hide)
-    )
-    (pin "1")
-    (pin "2")
-    (pin "3")
-    (pin "4")
-  )
-  (symbol (lib_id "synermycha-electronics:WS2812B_2020") (at 214.63 102.87 0) (unit 1)
-    (in_bom yes) (on_board yes)
-    (property "Reference" "D22" (id 0) (at 217.17 96.52 0)
-      (effects (font (size 1.27 1.27)) (justify left))
-    )
-    (property "Value" "WS2812B_2020" (id 1) (at 207.01 93.98 0)
-      (effects (font (size 1.27 1.27)) (justify left))
-    )
-    (property "Footprint" "WS2812-2020:WS28122020" (id 2) (at 215.9 110.49 0)
-      (effects (font (size 1.27 1.27)) (justify left top) hide)
-    )
-    (property "Datasheet" "https://cdn-shop.adafruit.com/datasheets/WS2812B.pdf" (id 3) (at 217.17 112.395 0)
-      (effects (font (size 1.27 1.27)) (justify left top) hide)
-    )
-    (pin "1")
-    (pin "2")
-    (pin "3")
-    (pin "4")
-  )
-  (symbol (lib_id "synermycha-electronics:WS2812B_2020") (at 123.19 102.87 0) (unit 1)
-    (in_bom yes) (on_board yes)
-    (property "Reference" "D20" (id 0) (at 125.73 96.52 0)
-      (effects (font (size 1.27 1.27)) (justify left))
-    )
-    (property "Value" "WS2812B_2020" (id 1) (at 115.57 93.98 0)
-      (effects (font (size 1.27 1.27)) (justify left))
-    )
-    (property "Footprint" "WS2812-2020:WS28122020" (id 2) (at 124.46 110.49 0)
-      (effects (font (size 1.27 1.27)) (justify left top) hide)
-    )
-    (property "Datasheet" "https://cdn-shop.adafruit.com/datasheets/WS2812B.pdf" (id 3) (at 125.73 112.395 0)
-      (effects (font (size 1.27 1.27)) (justify left top) hide)
-    )
-    (pin "1")
-    (pin "2")
-    (pin "3")
-    (pin "4")
-  )
 )
