File: test-points.kicad_sch (KiCad schematic)
At the start: 12 parts

Commit message: Clear test points
Parts:
- removed TP1, TP10, TP11, TP12, TP2, TP3, TP4, TP5, TP6, TP7, TP8, TP9: TestPoint, TestPoint:TestPoint_Pad_D1.5mm, symbol Connector:TestPoint
