File: as5045b_board/as5045b_board.kicad_pcb (KiCad board)
At the start: 4 copper layers, 21.8 x 12 mm, 20 parts, among them J1 Conn_01x04, J2 Conn_01x04, U1 AS5304, U2 AS5304

Commit message: Czyszczenie
Usunięto linie 5V oraz 2V8. Poprawiono symbol dla diody RGB
Parts:
- moved R6 5.08 mm to (-0.33, 7.27)
- moved R2 5.00 mm to (4.75, 7.25)
- moved R5 2.05 mm to (1.20, 7.75), turned to 180 degrees
- moved R1 2.00 mm to (3.25, 7.75), turned to 0 degrees
- moved R11 0.05 mm to (1.20, 6.75)
- turned J1 to 0 degrees
- turned U1 to 0 degrees
Connections:
- R11 pad 2: Net-(R1-Pad1) -> Net-(R11-Pad2)
- R5 pad 1: Net-(R5-Pad1) -> Net-(R11-Pad2)
- R9 pad 2: Net-(R5-Pad1) -> Net-(R1-Pad1)
- U1 pad 2: Net-(R5-Pad1) -> Net-(R1-Pad1)
- U1 pad 20: (no net) -> GND
- U1 pad 4: Net-(R1-Pad1) -> Net-(R11-Pad2)
- U2 pad 20: (no net) -> GND
Routing:
- net Net-(R11-Pad2): track 0.00 -> 10.6 mm
- net +5V: track 56.6 -> 62.1 mm, vias 11 -> 13
- net Net-(R1-Pad1): track 5.82 -> 10.9 mm
- net Net-(J1-Pad3): track 4.08 -> 8.48 mm
- net GND: track 62.4 -> 58.0 mm, vias 13 -> 12
- net Net-(R5-Pad1): track 4.10 -> 0.00 mm
