File: as5045b_board/as5045b_board.kicad_pcb (KiCad board)
At the start: 4 copper layers, 22 x 12 mm, 21 parts, among them J1 Conn_01x04, J2 Conn_01x04, U1 AS5304, U2 AS5304, U3 LTC3221

Commit message: Encoders update
Parts:
- removed C4: 10uF, Capacitor_SMD:C_0603_1608Metric
- removed R10, R12: DNP, Resistor_SMD:R_0402_1005Metric
- added C7: 2.2uF, Capacitor_SMD:C_0603_1608Metric, F.Cu at (-5.70, 6.50)
- added C8: 1uF, Capacitor_SMD:C_0402_1005Metric, F.Cu at (-5.50, 2.30)
- added C9: 4.7uF, Capacitor_SMD:C_0603_1608Metric, F.Cu at (-7.20, 3.90)
- added U4: LTC3221, Package_DFN_QFN:DFN-6-1EP_2x2mm_P0.5mm_EP0.61x1.42mm, F.Cu at (-5.40, 4.30)
- moved U2 191.8 mm to (-7.50, -1.55)
- moved C3 191.6 mm to (4.40, 4.00)
- moved C5 191.6 mm to (2.90, 6.50)
- moved J1 191.6 mm to (6.62, 6.45), turned to 180 degrees
- moved J2 191.6 mm to (-9.40, 6.45)
- moved R1 191.6 mm to (7.60, 4.20)
- moved R2 191.6 mm to (8.60, 4.20)
- moved R5 191.6 mm to (6.60, 4.20)
- moved R6 191.6 mm to (5.60, 4.20)
- moved C2 191.6 mm to (0.80, 2.30)
- moved C6 191.6 mm to (2.70, 2.30)
- moved U3 191.6 mm to (2.60, 4.30)
- moved U1 191.5 mm to (4.70, -1.55), turned to 180 degrees
- moved R3 191.4 mm to (-9.40, 4.20), turned to 270 degrees
- moved R7 191.3 mm to (-10.4, 4.20), turned to 270 degrees
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Connections:
- J2 pad 1: +5V -> Net-(C7-Pad1)
- R1 pad 2: Net-(J1-Pad4) -> Net-(J1-Pad3)
- R2 pad 1: Net-(J1-Pad4) -> Net-(J1-Pad3)
- R5 pad 2: Net-(J1-Pad3) -> Net-(J1-Pad4)
- R6 pad 1: Net-(J1-Pad3) -> Net-(J1-Pad4)
Routing:
- net GND: track 38.9 -> 2.71 mm, vias 14 -> 13
- net +5V: track 37.1 -> 10.6 mm
- net Net-(C7-Pad1): track 0.00 -> 11.4 mm, vias 0 -> 3
- net Net-(R1-Pad1): track 11.4 -> 4.41 mm
- net Net-(C5-Pad1): track 7.53 -> 11.8 mm, vias 2 -> 3
- net Net-(R5-Pad1): track 8.89 -> 5.68 mm
- net Net-(J2-Pad4): track 5.49 -> 3.14 mm
- net Net-(C8-Pad2): track 0.00 -> 1.32 mm
- net Net-(C8-Pad1): track 0.00 -> 1.12 mm
- net Net-(R3-Pad1): track 9.92 -> 8.93 mm
- net Net-(J1-Pad3): track 3.03 -> 3.94 mm

Commit message: Dodano grafiki do płytek enkodera
Parts:
- added G***: LOGO, footprints:dickbutt, B.Cu at (-7.50, -0.50)
- added G***: LOGO, graphics:PinUpGirl_silk_screen_4.4x9.8mm, B.Cu at (5.00, 1.00)

Commit message: Zmiany przy składaniu zamówienia
Parts:
- added mouse-bite-2mm-slot: VAL**, footprints:mouse-bite-2mm-slot, F.Cu at (15.0, 1.25)
- added mouse-bite-2mm-slot: VAL**, footprints:mouse-bite-2mm-slot, F.Cu at (15.0, 3.50)
- added mouse-bite-2mm-slot: VAL**, footprints:mouse-bite-2mm-slot, F.Cu at (15.0, -0.25)
- added mouse-bite-2mm-slot: VAL**, footprints:mouse-bite-2mm-slot, F.Cu at (15.0, -2.50)
- moved C1 28.4 mm to (24.8, 1.60)
- moved C7 28.4 mm to (22.7, 5.80)
- moved C8 28.4 mm to (22.9, 1.60)
- moved C9 28.4 mm to (21.2, 3.20)
- moved G*** 28.4 mm to (20.9, -1.20)
- moved J2 28.4 mm to (19.0, 5.75)
- moved R3 28.4 mm to (19.0, 3.50)
- moved R4 28.4 mm to (20.0, 3.50)
- moved R7 28.4 mm to (18.0, 3.50)
- moved R8 28.4 mm to (17.0, 3.50)
- moved U2 28.4 mm to (20.9, -2.25)
- moved U4 28.4 mm to (23.0, 3.60)
- moved C2 4.46 mm to (5.20, 1.60)
- moved C3 4.46 mm to (8.80, 3.30)
- moved C5 4.46 mm to (7.30, 5.80)
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Other:
- outline, holes or cut-outs redrawn
