File: as5045b_board/as5045b_board.sch (KiCad schematic (older format))
At the start: 20 parts, among them J1 Conn_01x04, J2 Conn_01x04, U1 AS5304, U2 AS5304

Commit message: Zaktualizowano enkodery
Parts:
- removed C4: 10uF, Capacitor_SMD:C_0603_1608Metric, symbol Device:C_Small
- removed R10, R11, R12, R9: 10K, Resistor_SMD:R_0402_1005Metric, symbol Device:R_Small
- added C5, C7: 2.2uF, Capacitor_SMD:C_0603_1608Metric, symbol Device:C_Small
- added C6, C8: 1uF, Capacitor_SMD:C_0402_1005Metric, symbol Device:C_Small
- added C9: 4.7uF, Capacitor_SMD:C_0603_1608Metric, symbol Device:C_Small
- added U3, U4: LTC3221, Package_DFN_QFN:DFN-6-1EP_2x2mm_P0.5mm_EP0.61x1.42mm, symbol synermycha-electronics:LTC3221
- C3: value 10uF -> 4.7uF
- U1, U2: symbol ams:AS5304 -> as5045b_board-rescue:AS5304-ams
Connections:
- net +5V: now also C9.1, U3.6 (VOUT), U4.6 (VOUT); no longer J1.1 (Pin_1), J2.1 (Pin_1)
- net GND: now also U1.20 (~CS), U2.20 (~CS), C5.2, C7.2, C9.2, U3.4 (GND), U3.7 (GND), U4.4 (GND), U4.7 (GND)
- net at R5.2, R6.1: now also J1.4 (Pin_4); no longer J1.3 (Pin_3)
- net at R1.2, R2.1: now also J1.3 (Pin_3); no longer J1.4 (Pin_4)
- net at U1.2 (A): now also R1.1; no longer R5.1
- net at U1.4 (B): now also R5.1; no longer R1.1
- new net: C5.1, J1.1 (Pin_1), U3.3 (~SHDN), U3.5 (VIN)
- new net: C7.1, J2.1 (Pin_1), U4.3 (~SHDN), U4.5 (VIN)
- new net: C6.1, U3.1 (C+)
- new net: C6.2, U3.2 (C-)
- new net: C8.1, U4.1 (C+)
- new net: C8.2, U4.2 (C-)
Other:
- note added: "Note:\nPin 20 of AS5304 is connected manually\nto GND on PBC Layout Editor"
- moved on the sheet: C2, C3, J1, J2, R3, R4, R7, R8
